Commit message: Added simulation example where the simulator (pelvis fixed) takes CASSIE_INPUT (LCM) as it's input and outputs (CASSIE_STATE). This should ideally interface with the Dispatcher, but works for now as a demonstration.

File: examples/Cassie/urdf/cassie_fixed_springs.urdf (robot description, URDF)
Before this commit: robot cassie, 21 links, 20 joints
Joints:
- joint ankle_joint_left: type revolute -> fixed
- joint ankle_joint_right: type revolute -> fixed
- joint toe_left: type fixed -> revolute
- joint toe_right: type fixed -> revolute
