Commit message: Lots of progress on updates. Simulation to PD control workflow is now functioning with the correct URDF. However, the workflow assumes the PD mapping is fixed by input->velocity via the B matrix. The Cassie URDF doesn't quite work this way, as the toe motors are "really" controlling one of the passive joints via springs. Either generalize the PD workflow or change the URDF, as this might be confusing long-term.

File: examples/Cassie/urdf/cassie.urdf (robot description, URDF)
Before this commit: robot cassie, 21 links, 20 joints
Joints:
- removed joint knee_motor_left
- removed joint knee_motor_right
- added joint knee_left: type revolute, parent thigh_left, child knee_left, origin xyz=0.12 0 0.0045 rpy=0 0 0, axis 0 0 1, limit lower=-2.862 upper=-0.646 effort=300
- added joint knee_right: type revolute, parent thigh_right, child knee_right, origin xyz=0.12 0 -0.0045 rpy=0 0 0, axis 0 0 1, limit lower=-2.862 upper=-0.646 effort=300

File: examples/Cassie/urdf/cassie_fixed_springs.urdf (robot description, URDF)
Before this commit: robot cassie, 21 links, 20 joints
Joints:
- removed joint knee_motor_left
- removed joint knee_motor_right
- added joint knee_left: type revolute, parent thigh_left, child knee_left, origin xyz=0.12 0 0.0045 rpy=0 0 0, axis 0 0 1, limit lower=-2.862 upper=-0.646 effort=300
- added joint knee_right: type revolute, parent thigh_right, child knee_right, origin xyz=0.12 0 -0.0045 rpy=0 0 0, axis 0 0 1, limit lower=-2.862 upper=-0.646 effort=300
