Commit message: adding urdfs with nearly identical inertia values to mujoco xml without armature

File: examples/Cassie/urdf/cassie_agility.urdf (robot description, URDF)
Before this commit: robot cassie, 23 links, 22 joints
Links:
- added link achilles_rod_left, mass 0.1567
- added link achilles_rod_right, mass 0.1567
- link foot_crank_mass_left: mass 0.129 -> 0.1261
- link foot_crank_mass_right: mass 0.129 -> 0.1261
- link heel_spring_left: mass 0.1259 -> 0.126
- link heel_spring_right: mass 0.1259 -> 0.126
- link knee_spring_left: mass 0.1864 -> 0.186
- link knee_spring_right: mass 0.1864 -> 0.186
- link shin_left: mass 0.5771 -> 0.577
- link shin_right: mass 0.5771 -> 0.577
Joints:
- added joint achilles_rod__left: type fixed, parent hip_left, child achilles_rod_left, origin xyz=0 0 0.045
- added joint achilles_rod_right: type fixed, parent hip_right, child achilles_rod_right, origin xyz=0 0 -0.045
- joint foot_crank_mass_left: origin xyz=.055 0 .00776 -> xyz=.058 -0.034 .02275; parent toe_left -> tarsus_left
- joint foot_crank_mass_right: origin xyz=.055 0 -.00776 -> xyz=.058 -0.034 -.02275; parent toe_right -> tarsus_right
- joint plantar_rod_mass_left: origin xyz=.055 0 .00776 -> xyz=.055 0 -.00791; parent toe_left -> foot_crank_mass_left
- joint plantar_rod_mass_right: origin xyz=.055 0 -.00776 -> xyz=.055 0 .00791; parent toe_right -> foot_crank_mass_right
