Commit message: drake to mujoco conversion working now

File: examples/Cassie/urdf/cassie_foot_crank.urdf (robot description, URDF)
Before this commit: robot foot_crank, 4 links, 3 joints
Joints:
- joint foot_crank_left: limit lower=-0.393 upper=0.393 effort=300 -> lower=-2.8 upper=0 effort=300; origin xyz=.055 0 .00776 -> xyz=.058 -0.034 0.02275; parent toe_left -> tarsus_left
- joint plantar_rod_left: limit lower=-0.393 upper=0.393 effort=300 -> lower=0 upper=2.8 effort=300

Commit message: working on fixing IK solver for drake to mujoco conversion

File: examples/Cassie/urdf/cassie_foot_crank.urdf (robot description, URDF)
Before this commit: robot foot_crank, 4 links, 3 joints
Links:
- link foot_crank_left: geometry visual mesh filename=meshes/agility/foot_crank.obj
- link plantar_rod_left: geometry visual mesh filename=meshes/agility/plantar_rod.obj
