Commit message: fourbar constraints for cassie bullet sim complete - need to finish state mapping functions to test

File: examples/Cassie/urdf/cassie_full_model_bullet.urdf (robot description, URDF)
Before this commit: robot cassie, 37 links, 36 joints
Links:
- removed link achilles_heel_pitch_left
- removed link achilles_heel_pitch_right
- removed link achilles_heel_roll_left
- removed link achilles_heel_roll_right
- removed link plantar_foot_pitch_left
- removed link plantar_foot_pitch_right
- removed link plantar_foot_roll_left
- removed link plantar_foot_roll_right
Joints:
- removed joint achilles_heel_pitch_left
- removed joint achilles_heel_pitch_right
- removed joint achilles_heel_roll_left
- removed joint achilles_heel_roll_right
- removed joint plantar_foot_pitch_left
- removed joint plantar_foot_pitch_right
- removed joint plantar_foot_roll_left
- removed joint plantar_foot_roll_right

Commit message: finish urdf editing

File: examples/Cassie/urdf/cassie_full_model_bullet.urdf (robot description, URDF)
Before this commit: robot cassie, 29 links, 28 joints
Joints:
- removed joint toe_crank_left
- removed joint toe_crank_right
- added joint toe_ee_left: type revolute, parent tarsus_left, child toe_left, origin xyz=0.408 -0.040 0 rpy=0 0 0, axis 0 0 1, limit lower=-3.14 upper=3.14
- added joint toe_ee_right: type revolute, parent tarsus_right, child toe_right, origin xyz=0.408 -0.040 0 rpy=0 0 0, axis 0 0 1, limit lower=-3.14 upper=3.14
- joint toe_left: child toe_left -> foot_crank_link_left; limit lower=-3.14 upper=3.14 -> lower=-2.443 upper=-0.524 effort=300; origin xyz=0.408 -0.040 0 rpy=0 0 0 -> xyz=0.058 -0.034 0.02275 rpy=0 0 0
- joint toe_right: child toe_right -> foot_crank_link_right; limit lower=-3.14 upper=3.14 -> lower=-2.443 upper=-0.524 effort=300; origin xyz=0.408 -0.040 0 rpy=0 0 0 -> xyz=0.058 -0.034 -0.02275 rpy=0 0 0

Commit message: remaining ik work is to solve for joint angles of achilles hip joint

File: examples/Cassie/urdf/cassie_full_model_bullet.urdf (robot description, URDF)
Before this commit: robot cassie, 29 links, 28 joints
Links:
- link foot_crank_link_left: geometry visual mesh filename=meshes/toe-output-crank.obj
- link foot_crank_link_right: geometry visual mesh filename=meshes/toe-output-crank-r.obj

Commit message: nullet indexing fixes

File: examples/Cassie/urdf/cassie_full_model_bullet.urdf (robot description, URDF)
Before this commit: robot cassie, 29 links, 28 joints
Links:
- link toe_left: geometry collision sphere radius=0.001; collision sphere radius=0.001
- link toe_right: geometry collision sphere radius=0.001; collision sphere radius=0.001
