Commit message: add footstep z target from depth

File: examples/Cassie/urdf/cassie_v2_sc.urdf (robot description, URDF)
Before this commit: robot cassie, 23 links, 22 joints
Links:
- link pelvis: geometry collision sphere radius=0.2; visual mesh filename=meshes/pelvis.obj
- link shin_left: geometry collision cylinder length=0.4 radius=0.015; visual mesh filename=meshes/agility/left_shin.obj
- link shin_right: geometry collision cylinder length=0.4 radius=0.015; visual mesh filename=meshes/agility/right_shin.obj
- link tarsus_left: geometry collision cylinder length=0.4 radius=0.015; visual mesh filename=meshes/tarsus.obj
- link tarsus_right: geometry collision cylinder length=0.4 radius=0.015; visual mesh filename=meshes/tarsus-r.obj
- link toe_left: geometry collision box size=0.1 0.03 0.03; collision sphere radius=0.0
- link toe_right: geometry collision box size=0.1 0.03 0.03; collision sphere radius=0.0
