Commit message: working in drake and mujoco

File: examples/Cassie/urdf/cassie_v2_conservative.urdf (robot description, URDF)
Before this commit: robot cassie, 23 links, 22 joints
Joints:
- joint knee_left: limit lower=-2.862 upper=-0.646 effort=300 -> lower=-2.862 upper=-0.646 effort=195
- joint knee_right: limit lower=-2.862 upper=-0.646 effort=300 -> lower=-2.862 upper=-0.646 effort=195
- joint toe_left: limit lower=-2.0 upper=-0.74 effort=150 -> lower=-2.0 upper=-0.74 effort=50
- joint toe_right: limit lower=-2.0 upper=-0.74 effort=150 -> lower=-2.0 upper=-0.74 effort=50

Commit message: gain tuning, adding input limits

File: examples/Cassie/urdf/cassie_v2_conservative.urdf (robot description, URDF)
Before this commit: robot cassie, 23 links, 22 joints
Joints:
- joint hip_pitch_left: limit lower=0.2 upper=1.24 effort=300 -> lower=0.2 upper=1.24 effort=90
- joint hip_pitch_right: limit lower=0.2 upper=1.24 effort=300 -> lower=0.2 upper=1.24 effort=90
- joint hip_roll_left: limit lower=-0.05 upper=0.100 effort=300 -> lower=-0.05 upper=0.100 effort=90
- joint hip_roll_right: limit lower=-0.100 upper=0.05 effort=300 -> lower=-0.100 upper=0.05 effort=90
- joint hip_yaw_left: limit lower=0.0 upper=0.2 effort=300 -> lower=0.0 upper=0.2 effort=60
- joint hip_yaw_right: limit lower=-0.2 upper=0.0 effort=300 -> lower=-0.2 upper=0.0 effort=60
- joint knee_left: limit lower=-2.862 upper=-0.646 effort=195 -> lower=-2.862 upper=-0.646 effort=200
- joint knee_right: limit lower=-2.862 upper=-0.646 effort=195 -> lower=-2.862 upper=-0.646 effort=200
- joint toe_left: limit lower=-2.0 upper=-0.74 effort=50 -> lower=-2.0 upper=-0.74 effort=40
- joint toe_right: limit lower=-2.0 upper=-0.74 effort=50 -> lower=-2.0 upper=-0.74 effort=40

Commit message: changing some scaling

File: examples/Cassie/urdf/cassie_v2_conservative.urdf (robot description, URDF)
Before this commit: robot cassie, 23 links, 22 joints
Joints:
- joint toe_left: limit lower=-2.0 upper=-0.74 effort=40 -> lower=-2.0 upper=-0.74 effort=20
- joint toe_right: limit lower=-2.0 upper=-0.74 effort=40 -> lower=-2.0 upper=-0.74 effort=20

Commit message: relaxing toe actuator limits

File: examples/Cassie/urdf/cassie_v2_conservative.urdf (robot description, URDF)
Before this commit: robot cassie, 23 links, 22 joints
Joints:
- joint toe_left: limit lower=-2.0 upper=-0.74 effort=20 -> lower=-2.0 upper=-0.74 effort=40
- joint toe_right: limit lower=-2.0 upper=-0.74 effort=20 -> lower=-2.0 upper=-0.74 effort=40
