Commit message: lighting on drake visualizer looks weird still

File: examples/Cassie/urdf/cassie_v2_shells.urdf (robot description, URDF)
Before this commit: robot cassie, 23 links, 22 joints
Links:
- link heel_spring_left: geometry visual mesh filename=meshes/agility/heel-spring.obj
- link heel_spring_right: geometry visual mesh filename=meshes/agility/heel-spring.obj
- link toe_right: geometry collision sphere radius=0.0; collision sphere radius=0.0

Commit message: working on making visualization scripts in python

File: examples/Cassie/urdf/cassie_v2_shells.urdf (robot description, URDF)
Before this commit: robot cassie, 23 links, 22 joints
Links:
- link tarsus_right: geometry visual mesh filename=meshes/agility/tarsus.obj scale=-1 -1 -1
