Commit message: Simulation with both achilles and plantar rods now runs. Set a reasonable initial guess in the simulation as well.

File: examples/Cassie/urdf/cassie_v2.urdf (robot description, URDF)
Before this commit: robot cassie, 27 links, 26 joints
Links:
- added link achilles_heel_roll_left
- added link achilles_heel_roll_right
- added link plantar_crank_pitch_left
- added link plantar_crank_pitch_right
- added link plantar_foot_pitch_left
- added link plantar_foot_pitch_right
- added link plantar_foot_roll_left
- added link plantar_foot_roll_right
- added link plantar_rod_left, mass 0.1186; visual mesh filename=meshes/plantar-rod.obj
- added link plantar_rod_right, mass 0.1186; visual mesh filename=meshes/plantar-rod.obj
- link heel_spring_left: geometry visual mesh filename=meshes/heel-spring.obj
Joints:
- added joint achilles_heel_roll_left: type revolute, parent achilles_rod_left, child achilles_heel_roll_left, origin xyz=.5012 0 0, axis 1 0 0, limit lower=-20 upper=20
- added joint achilles_heel_roll_right: type revolute, parent achilles_rod_right, child achilles_heel_roll_right, origin xyz=.5012 0 0, axis 1 0 0, limit lower=-3.14 upper=3.14
- added joint plantar_crank_left: type revolute, parent foot_crank_link_left, child plantar_crank_pitch_left, origin xyz=0.055  0  -.00791 rpy=0 0 0, axis 0 1 0, limit lower=-3.14 upper=3.14
- added joint plantar_crank_pitch_left: type revolute, parent plantar_crank_pitch_left, child plantar_rod_left, axis 0 0 1, limit lower=-3.14 upper=3.14
- added joint plantar_crank_pitch_right: type revolute, parent plantar_crank_pitch_right, child plantar_rod_right, axis 0 0 1, limit lower=-3.14 upper=3.14
- added joint plantar_crank_right: type revolute, parent foot_crank_link_right, child plantar_crank_pitch_right, origin xyz=0.055  0  .00791 rpy=0 0 0, axis 0 1 0, limit lower=-3.14 upper=3.14
- added joint plantar_foot_pitch_left: type revolute, parent plantar_foot_roll_left, child plantar_foot_pitch_left, origin xyz=0 0 0, axis 0 1 0, limit lower=-3.14 upper=3.14
- added joint plantar_foot_pitch_right: type revolute, parent plantar_foot_roll_right, child plantar_foot_pitch_right, origin xyz=0 0 0, axis 0 1 0, limit lower=-3.14 upper=3.14
- added joint plantar_foot_roll_left: type revolute, parent plantar_rod_left, child plantar_foot_roll_left, origin xyz=.35012 0 0, axis 1 0 0, limit lower=-3.14 upper=3.14
- added joint plantar_foot_roll_right: type revolute, parent plantar_rod_right, child plantar_foot_roll_right, origin xyz=.35012 0 0, axis 1 0 0, limit lower=-3.14 upper=3.14
- joint achilles_heel_pitch_left: origin xyz=.5012 0 0 -> xyz=0 0 0; parent achilles_rod_left -> achilles_heel_roll_left
- joint achilles_heel_pitch_right: origin xyz=.5012 0 0 -> xyz=0 0 0; parent achilles_rod_right -> achilles_heel_roll_right
- joint toe_crank_left: type fixed -> revolute
- joint toe_crank_right: type fixed -> revolute
- joint toe_left: limit lower=-2.443 upper=-0.524 effort=300 -> lower=-3.14 upper=3.14
- joint toe_right: limit lower=-2.443 upper=-0.524 effort=300 -> lower=-3.14 upper=3.14

Commit message: tuning in drake with correct motor model

File: examples/Cassie/urdf/cassie_v2.urdf (robot description, URDF)
Before this commit: robot cassie, 23 links, 22 joints
Joints:
- joint hip_pitch_left: limit lower=-0.873 upper=1.396 effort=300 -> lower=-0.873 upper=1.396 effort=195.2
- joint hip_pitch_right: limit lower=-0.873 upper=1.396 effort=300 -> lower=-0.873 upper=1.396 effort=195.2
- joint hip_roll_left: limit lower=-0.262 upper=0.393 effort=300 -> lower=-0.262 upper=0.393 effort=112.5
- joint hip_roll_right: limit lower=-0.393 upper=0.262 effort=300 -> lower=-0.393 upper=0.262 effort=112.5
- joint hip_yaw_left: limit lower=-0.393 upper=0.393 effort=300 -> lower=-0.393 upper=0.393 effort=112.5
- joint hip_yaw_right: limit lower=-0.393 upper=0.393 effort=300 -> lower=-0.393 upper=0.393 effort=112.5
- joint knee_left: limit lower=-2.862 upper=-0.646 effort=300 -> lower=-2.862 upper=-0.646 effort=195.2
- joint knee_right: limit lower=-2.862 upper=-0.646 effort=300 -> lower=-2.862 upper=-0.646 effort=195.2
- joint toe_left: limit lower=-2.8 upper=0 effort=300 -> lower=-2.8 upper=0 effort=45
- joint toe_right: limit lower=-2.8 upper=0 effort=300 -> lower=-2.8 upper=0 effort=45

File: examples/Cassie/urdf/cassie_v2_conservative.urdf (robot description, URDF)
Before this commit: robot cassie, 23 links, 22 joints
Joints:
- joint knee_left: limit lower=-2.862 upper=-0.646 effort=200 -> lower=-2.862 upper=-0.646 effort=195.2
- joint knee_right: limit lower=-2.862 upper=-0.646 effort=200 -> lower=-2.862 upper=-0.646 effort=195.2

Commit message: add collision geometries, except to thighs

File: examples/Cassie/urdf/cassie_v2.urdf (robot description, URDF)
Before this commit: robot cassie, 23 links, 22 joints
Links:
- link pelvis: geometry collision sphere radius=0.2; visual mesh filename=meshes/pelvis.obj
- link shin_left: geometry collision cylinder length=0.4 radius=0.015; visual cylinder length=0.4 radius=0.015
- link shin_right: geometry collision cylinder length=0.4 radius=0.015; visual cylinder length=0.4 radius=0.015
- link tarsus_left: geometry collision cylinder length=0.4 radius=0.015; visual cylinder length=0.4 radius=0.015
- link tarsus_right: geometry collision cylinder length=0.4 radius=0.015; visual cylinder length=0.4 radius=0.015
- link toe_left: geometry collision box size=0.1 0.03 0.03; collision sphere radius=0.0
- link toe_right: geometry collision box size=0.1 0.03 0.03; collision sphere radius=0.0

Commit message: lots of changes, added environment, rough terrain testing script, and ability to pass in heightmap variance

File: examples/Cassie/urdf/cassie_v2.urdf (robot description, URDF)
Before this commit: robot cassie, 23 links, 22 joints
Links:
- link pelvis: geometry collision sphere radius=0.2; visual mesh filename=meshes/pelvis.obj

Commit message: updating contact scheduler

File: examples/Cassie/urdf/cassie_v2.urdf (robot description, URDF)
Before this commit: robot cassie, 23 links, 22 joints
Joints:
- joint knee_joint_left: limit lower=-.35 upper=0.35 -> lower=-.35 upper=0.035
- joint knee_joint_right: limit lower=-.35 upper=0.35 -> lower=-.35 upper=0.035

Commit message: sim changes

File: examples/Cassie/urdf/cassie_v2.urdf (robot description, URDF)
Before this commit: robot cassie, 23 links, 22 joints
Links:
- link toe_left: geometry collision sphere radius=0.01; collision sphere radius=0.01
- link toe_right: geometry collision sphere radius=0.01; collision sphere radius=0.01

Commit message: gltf meshes

File: examples/Cassie/urdf/cassie_v2.urdf (robot description, URDF)
Before this commit: robot cassie, 23 links, 22 joints
Links:
- link heel_spring_left: geometry visual mesh filename=meshes/heel-spring.gltf
- link heel_spring_right: geometry visual mesh filename=meshes/heel-spring.gltf
- link hip_left: geometry visual mesh filename=meshes/agility/left_hip.gltf
- link hip_right: geometry visual mesh filename=meshes/agility/right_hip.gltf
- link knee_left: geometry visual mesh filename=meshes/knee-output.gltf
- link knee_right: geometry visual mesh filename=meshes/knee-output-r.gltf
- link knee_spring_left: geometry visual mesh filename=meshes/knee-spring.gltf
- link knee_spring_right: geometry visual mesh filename=meshes/knee-spring.gltf
- link pelvis: geometry visual mesh filename=meshes/pelvis.gltf
- link shin_left: geometry visual mesh filename=meshes/agility/left_shin.gltf
- link shin_right: geometry visual mesh filename=meshes/agility/right_shin.gltf
- link tarsus_left: geometry visual mesh filename=meshes/tarsus.gltf
- link tarsus_right: geometry visual mesh filename=meshes/tarsus-r.gltf
- link thigh_left: geometry visual mesh filename=meshes/agility/left_thigh.gltf
- link thigh_right: geometry visual mesh filename=meshes/agility/right_thigh.gltf
- link toe_left: geometry collision sphere radius=0.01; collision sphere radius=0.01
- link toe_right: geometry collision sphere radius=0.01; collision sphere radius=0.01
- link yaw_left: geometry visual mesh filename=meshes/agility/left_yaw.gltf
- link yaw_right: geometry visual mesh filename=meshes/agility/right_yaw.gltf

Commit message: add normals to objs and remove gltf

File: examples/Cassie/urdf/cassie_v2.urdf (robot description, URDF)
Before this commit: robot cassie, 23 links, 22 joints
Links:
- link heel_spring_left: geometry visual mesh filename=meshes/heel-spring.obj
- link heel_spring_right: geometry visual mesh filename=meshes/heel-spring.obj
- link hip_left: geometry visual mesh filename=meshes/agility/left_hip.obj
- link hip_right: geometry visual mesh filename=meshes/agility/right_hip.obj
- link knee_left: geometry visual mesh filename=meshes/knee-output.obj
- link knee_right: geometry visual mesh filename=meshes/knee-output-r.obj
- link knee_spring_left: geometry visual mesh filename=meshes/knee-spring.obj
- link knee_spring_right: geometry visual mesh filename=meshes/knee-spring.obj
- link pelvis: geometry visual mesh filename=meshes/pelvis.obj
- link shin_left: geometry visual mesh filename=meshes/agility/left_shin.obj
- link shin_right: geometry visual mesh filename=meshes/agility/right_shin.obj
- link tarsus_left: geometry visual mesh filename=meshes/tarsus.obj
- link tarsus_right: geometry visual mesh filename=meshes/tarsus-r.obj
- link thigh_left: geometry visual mesh filename=meshes/agility/left_thigh.obj
- link thigh_right: geometry visual mesh filename=meshes/agility/right_thigh.obj
- link toe_left: geometry collision sphere radius=0.01; collision sphere radius=0.01
- link toe_right: geometry collision sphere radius=0.01; collision sphere radius=0.01
- link yaw_left: geometry visual mesh filename=meshes/agility/left_yaw.obj
- link yaw_right: geometry visual mesh filename=meshes/agility/right_yaw.obj

Commit message: some file deletions

File: examples/Cassie/urdf/cassie_v2.urdf (robot description, URDF)
Before this commit: robot cassie, 23 links, 22 joints
Links:
- link toe_left: geometry collision sphere radius=0.0; collision sphere radius=0.0
- link toe_right: geometry collision sphere radius=0.0; collision sphere radius=0.0

Commit message: update cassie urdf for lighter battery

File: examples/Cassie/urdf/cassie_v2.urdf (robot description, URDF)
Before this commit: robot cassie, 23 links, 22 joints
Links:
- link pelvis: mass 10.33 -> 9.33

File: examples/Cassie/urdf/cassie_v2_conservative.urdf (robot description, URDF)
Before this commit: robot cassie, 23 links, 22 joints
Links:
- link pelvis: mass 10.33 -> 9.33

File: examples/Cassie/urdf/cassie_v2_self_collision.urdf (robot description, URDF)
Before this commit: robot cassie, 23 links, 22 joints
Links:
- link pelvis: mass 10.33 -> 9.33
