Commit message: reset if foot stuck

File: examples/Cassie/urdf/cassie_v2_self_collision.urdf (robot description, URDF)
Before this commit: robot cassie, 23 links, 22 joints
Links:
- link toe_left: geometry collision box size=0.1 0.03 0.03; collision sphere radius=0.0
- link toe_right: geometry collision box size=0.1 0.03 0.03; collision sphere radius=0.0

Commit message: update joint limits in stepnet sim plant

File: examples/Cassie/urdf/cassie_v2_self_collision.urdf (robot description, URDF)
Before this commit: robot cassie, 23 links, 22 joints
Joints:
- joint ankle_spring_joint_left: limit lower=-1 upper=0.5 -> lower=-.1 upper=0.1
- joint ankle_spring_joint_right: limit lower=-1 upper=0.5 -> lower=-.1 upper=0.1
- joint hip_pitch_left: limit lower=-0.873 upper=1.396 effort=300 -> lower=0.2 upper=1.24 effort=90
- joint hip_pitch_right: limit lower=-0.873 upper=1.396 effort=300 -> lower=0.2 upper=1.24 effort=90
- joint hip_roll_left: limit lower=-0.262 upper=0.393 effort=300 -> lower=-0.05 upper=0.100 effort=90
- joint hip_roll_right: limit lower=-0.393 upper=0.262 effort=300 -> lower=-0.100 upper=0.05 effort=90
- joint hip_yaw_left: limit lower=-0.393 upper=0.393 effort=300 -> lower=0.0 upper=0.2 effort=60
- joint hip_yaw_right: limit lower=-0.393 upper=0.393 effort=300 -> lower=-0.2 upper=0.0 effort=60
- joint knee_joint_left: limit lower=-.35 upper=0.35 -> lower=-.1 upper=0.075
- joint knee_joint_right: limit lower=-.35 upper=0.35 -> lower=-.1 upper=0.075
- joint knee_left: limit lower=-2.862 upper=-0.646 effort=300 -> lower=-2.862 upper=-0.646 effort=200
- joint knee_right: limit lower=-2.862 upper=-0.646 effort=300 -> lower=-2.862 upper=-0.646 effort=200
- joint toe_left: limit lower=-2.8 upper=0 effort=300 -> lower=-2.0 upper=-0.74 effort=40
- joint toe_right: limit lower=-2.8 upper=0 effort=300 -> lower=-2.0 upper=-0.74 effort=40

Commit message: change the timing update logic and remove running cost on y-tracking to avoid weird effects

File: examples/Cassie/urdf/cassie_v2_self_collision.urdf (robot description, URDF)
Before this commit: robot cassie, 23 links, 22 joints
Joints:
- joint hip_roll_left: limit lower=-0.05 upper=0.100 effort=90 -> lower=-0.05 upper=0.20 effort=90
- joint hip_roll_right: limit lower=-0.100 upper=0.05 effort=90 -> lower=-0.20 upper=0.05 effort=90

Commit message: expand hip roll joint limits to match cassie doc, fix aspects of gait generation

File: examples/Cassie/urdf/cassie_v2_self_collision.urdf (robot description, URDF)
Before this commit: robot cassie, 23 links, 22 joints
Links:
- link toe_left: geometry collision box size=0.1 0.03 0.03; collision sphere radius=0.0
- link toe_right: geometry collision box size=0.1 0.03 0.03; collision sphere radius=0.0
Joints:
- joint hip_roll_left: limit lower=-0.05 upper=0.20 effort=90 -> lower=-0.34 upper=0.34 effort=90
- joint hip_roll_right: limit lower=-0.20 upper=0.05 effort=90 -> lower=-0.34 upper=0.34 effort=90

Commit message: update joint limits to match hardware

File: examples/Cassie/urdf/cassie_v2_self_collision.urdf (robot description, URDF)
Before this commit: robot cassie, 23 links, 22 joints
Joints:
- joint hip_roll_left: limit lower=-0.34 upper=0.34 effort=90 -> lower=-0.11 upper=0.2 effort=90
- joint hip_roll_right: limit lower=-0.34 upper=0.34 effort=90 -> lower=-0.11 upper=0.2 effort=90
- joint hip_yaw_left: limit lower=0.0 upper=0.2 effort=60 -> lower=-0.235 upper=0.235 effort=60
- joint hip_yaw_right: limit lower=-0.2 upper=0.0 effort=60 -> lower=-0.235 upper=0.235 effort=60

Commit message: update contact spheres

File: examples/Cassie/urdf/cassie_v2_self_collision.urdf (robot description, URDF)
Before this commit: robot cassie, 23 links, 22 joints
Links:
- link toe_left: geometry collision box size=0.1 0.03 0.03; collision sphere radius=0.001
- link toe_right: geometry collision box size=0.1 0.03 0.03; collision sphere radius=0.001

Commit message: experiment working

File: examples/Cassie/urdf/cassie_v2_self_collision.urdf (robot description, URDF)
Before this commit: robot cassie, 23 links, 22 joints
Links:
- link pelvis: geometry collision sphere radius=0.2; visual mesh filename=meshes/agility/pelvis.obj
- link shin_left: geometry collision cylinder length=0.4 radius=0.025; visual mesh filename=meshes/agility/shin.obj
- link shin_right: geometry collision cylinder length=0.4 radius=0.025; visual mesh filename=meshes/agility/shin.obj scale=-1 -1 -1
- link tarsus_left: geometry collision cylinder length=0.4 radius=0.025; visual mesh filename=meshes/agility/tarsus.obj
- link tarsus_right: geometry collision cylinder length=0.4 radius=0.025; visual mesh filename=meshes/agility/tarsus.obj scale=-1 -1 -1
- link thigh_left: geometry visual mesh filename=meshes/agility/hip-pitch.obj
- link thigh_right: geometry visual mesh filename=meshes/agility/hip-pitch.obj scale=-1 -1 -1

Commit message: adjust urdf

File: examples/Cassie/urdf/cassie_v2_self_collision.urdf (robot description, URDF)
Before this commit: robot cassie, 23 links, 22 joints
Links:
- link toe_left: geometry collision box size=0.17 0.01 0.01; collision sphere radius=0.001
- link toe_right: geometry collision box size=0.17 0.01 0.01; collision sphere radius=0.001

Commit message: sim tuning

File: examples/Cassie/urdf/cassie_v2_self_collision.urdf (robot description, URDF)
Before this commit: robot cassie, 23 links, 22 joints
Links:
- link toe_left: geometry collision box size=0.15 0.001 0.001; collision sphere radius=0.0025
- link toe_right: geometry collision box size=0.15 0.01 0.01; collision sphere radius=0.0025

Commit message: upadtes to work w new perception stack and do MPC

File: examples/Cassie/urdf/cassie_v2_self_collision.urdf (robot description, URDF)
Before this commit: robot cassie, 23 links, 22 joints
Links:
- link pelvis: mass 10.33 -> 9.33
- link toe_left: geometry collision box size=0.15 0.001 0.001; collision sphere radius=0.0025
- link toe_right: geometry collision box size=0.15 0.01 0.01; collision sphere radius=0.0025

Commit message: tune sim experiments with vision in the loop and self collisions

File: examples/Cassie/urdf/cassie_v2_self_collision.urdf (robot description, URDF)
Before this commit: robot cassie, 23 links, 22 joints
Links:
- link toe_left: geometry collision box size=0.15 0.01 0.01; collision sphere radius=0.001
- link toe_right: geometry collision box size=0.15 0.01 0.01; collision sphere radius=0.001

Commit message: lots of cf-mpfc tests and progress

File: examples/Cassie/urdf/cassie_v2_self_collision.urdf (robot description, URDF)
Before this commit: robot cassie, 23 links, 22 joints
Links:
- link toe_left: geometry collision box size=0.15 0.001 0.001; visual box size=0.15 0.01 0.01
- link toe_right: geometry collision box size=0.15 0.01 0.01; visual box size=0.15 0.01 0.01
