Commit message: The code compiles but the controller is unstable

File: examples/PlanarWalker/PlanarWalkerWithTorsoAndFeet.urdf (robot description, URDF)
Before this commit: robot KneedCompassGaitWithFeet, 15 links, 14 joints
Links:
- added link left_foot_mass, mass 0.5; visual sphere radius=0.025
- added link right_foot_mass, mass 0.5; visual sphere radius=0.025
Joints:
- added joint left_foot_mass_weld: type fixed, parent left_foot, child left_foot_mass
- added joint right_foot_mass_weld: type fixed, parent right_foot, child right_foot_mass
- joint left_ankle: type revolute -> continuous
- joint right_ankle: type revolute -> continuous
- joint right_knee_pin: type revolute -> continuous

Commit message: Working zero step OSC
Zero step of OSC is working well and the tracking performance is good.
FSM is not tested in this commit.

File: examples/PlanarWalker/PlanarWalkerWithTorsoAndFeet.urdf (robot description, URDF)
Before this commit: robot KneedCompassGaitWithFeet, 17 links, 16 joints
Links:
- link left_foot: geometry collision sphere radius=0; collision sphere radius=0
- link left_lower_leg: geometry visual cylinder length=0.5 radius=0.0075
- link right_foot: geometry collision sphere radius=0; collision sphere radius=0
- link right_lower_leg: geometry visual cylinder length=0.5 radius=0.0075
