Commit message: Partially working safe trajectory tracking

File: examples/PlanarWalker/PlanarWalkerWithTorso.urdf (robot description, URDF)
Before this commit: robot KneedCompassGait, 13 links, 12 joints
Links:
- added link left_foot; collision sphere radius=0; collision sphere radius=0
- added link left_foot_mass, mass 0.5; visual sphere radius=0.025
- added link right_foot; collision sphere radius=0; collision sphere radius=0
- added link right_foot_mass, mass 0.5; visual sphere radius=0.025
- link left_lower_leg: geometry visual cylinder length=0.5 radius=0.0075
- link right_lower_leg: geometry visual cylinder length=0.5 radius=0.0075
Joints:
- added joint left_ankle: type continuous, parent left_lower_leg, child left_foot, origin xyz=0 0 -0.5 rpy=0 1.57 0, axis 0 1 0, limit lower=0 effort=100
- added joint left_foot_mass_weld: type fixed, parent left_foot, child left_foot_mass
- added joint right_ankle: type continuous, parent right_lower_leg, child right_foot, origin xyz=0 0 -0.5 rpy=0 1.57 0, axis 0 1 0, limit lower=0 effort=100
- added joint right_foot_mass_weld: type fixed, parent right_foot, child right_foot_mass
- joint right_knee_pin: type revolute -> continuous

File: examples/PlanarWalker/PlanarWalkerWithTorsoAndFeet.urdf (robot description, URDF)
Before this commit: robot KneedCompassGaitWithFeet, 17 links, 16 joints
Joints:
- joint left_ankle: limit lower=0 effort=100 -> lower=-100 effort=100
- joint left_knee_pin: limit lower=0 effort=100 -> lower=-100 effort=100
- joint right_ankle: limit lower=0 effort=100 -> lower=-100 effort=100
- joint right_knee_pin: limit lower=0 effort=100 -> lower=-100 effort=100

Commit message: planar walker dircon with torso

File: examples/PlanarWalker/PlanarWalkerWithTorso.urdf (robot description, URDF)
Before this commit: robot KneedCompassGait, 13 links, 12 joints
Links:
- link left_lower_leg_mass: mass 2.5 -> 2.0
- link right_lower_leg_mass: mass 2.5 -> 2.0
- link torso_mass: mass 10 -> 20

Commit message: Should reliably not have an infeasible mpc qp - still much to debug

File: examples/PlanarWalker/PlanarWalkerWithTorso.urdf (robot description, URDF)
Before this commit: robot KneedCompassGait, 13 links, 12 joints
Links:
- link torso_mass: mass 20 -> 21

Commit message: changed urdf, added debug features too koopman mpc, fixed ordering of lcm traj, and fixed laoding of dynamics matrices

File: examples/PlanarWalker/PlanarWalkerWithTorso.urdf (robot description, URDF)
Before this commit: robot KneedCompassGait, 13 links, 12 joints
Links:
- link left_lower_leg_mass: mass 2.0 -> 1
- link left_upper_leg_mass: mass 2.5 -> 1
- link right_lower_leg_mass: mass 2.0 -> 1
- link right_upper_leg_mass: mass 2.5 -> 1
- link torso_mass: mass 21 -> 26

Commit message: things appear to at least run as they should. Not walking yet. Need to check tracking and foot splines

File: examples/PlanarWalker/PlanarWalkerWithTorso.urdf (robot description, URDF)
Before this commit: robot KneedCompassGait, 13 links, 12 joints
Links:
- link left_lower_leg_mass: mass 1 -> 2
- link left_upper_leg_mass: mass 1 -> 2
- link right_lower_leg_mass: mass 1 -> 2
- link right_upper_leg_mass: mass 1 -> 2
- link torso_mass: mass 26 -> 22

Commit message: Adding plotting scripts

File: examples/PlanarWalker/PlanarWalkerWithTorso.urdf (robot description, URDF)
Before this commit: robot KneedCompassGait, 13 links, 12 joints
Links:
- link left_lower_leg_mass: mass 2 -> 1
- link left_upper_leg_mass: mass 2 -> 1
- link right_lower_leg_mass: mass 2 -> 1
- link right_upper_leg_mass: mass 2 -> 1
- link torso_mass: mass 22 -> 29

Commit message: added soft constraints - need to debug reachability

File: examples/PlanarWalker/PlanarWalkerWithTorso.urdf (robot description, URDF)
Before this commit: robot KneedCompassGait, 13 links, 12 joints
Links:
- link left_lower_leg_mass: mass 1 -> 0.25
- link left_upper_leg_mass: mass 1 -> 0.25
- link right_lower_leg_mass: mass 1 -> 0.25
- link right_upper_leg_mass: mass 1 -> 0.25
Joints:
- joint left_hip_pin: limit (none) -> effort=500
- joint left_knee_pin: limit lower=0 effort=100 -> lower=0 effort=400
- joint right_hip_pin: limit (none) -> effort=500
- joint right_knee_pin: limit lower=0 effort=100 -> lower=0 effort=400

Commit message: pushing most recent tweaks

File: examples/PlanarWalker/PlanarWalkerWithTorso.urdf (robot description, URDF)
Before this commit: robot KneedCompassGait, 13 links, 12 joints
Joints:
- joint torso_mass_weld: origin xyz=0 0 0.3 -> xyz=0 0 0

Commit message: turned kinematic reachability into a soft constraint

File: examples/PlanarWalker/PlanarWalkerWithTorso.urdf (robot description, URDF)
Before this commit: robot KneedCompassGait, 13 links, 12 joints
Links:
- link left_lower_leg_mass: mass 0.25 -> 1
- link left_upper_leg_mass: mass 0.25 -> 2
- link right_lower_leg_mass: mass 0.25 -> 1
- link right_upper_leg_mass: mass 0.25 -> 2
- link torso_mass: mass 29 -> 26
Joints:
- joint torso_mass_weld: origin xyz=0 0 0 -> xyz=0 0 0.15

Commit message: Fixed world point evaluators for osc

File: examples/PlanarWalker/PlanarWalkerWithTorso.urdf (robot description, URDF)
Before this commit: robot KneedCompassGait, 13 links, 12 joints
Links:
- link torso_mass: mass 26 -> 30
Joints:
- joint torso_mass_weld: origin xyz=0 0 0.15 -> xyz=0 0 0.3

Commit message: still deugging mpc :(

File: examples/PlanarWalker/PlanarWalkerWithTorso.urdf (robot description, URDF)
Before this commit: robot KneedCompassGait, 13 links, 12 joints
Links:
- link left_lower_leg_mass: mass 1 -> .125
- link left_upper_leg_mass: mass 2 -> 0.125
- link right_lower_leg_mass: mass 1 -> .125
- link right_upper_leg_mass: mass 2 -> .125

Commit message: fixed rotation axis for x-z plane and added fixed point solver for initial condition. Updated initial state force value to more closely match reality

File: examples/PlanarWalker/PlanarWalkerWithTorso.urdf (robot description, URDF)
Before this commit: robot KneedCompassGait, 13 links, 12 joints
Joints:
- joint planar_roty: axis 0 1 0 -> 0 -1 0

Commit message: Changed force calcs, koopman mpc seems to work ok in a few circumstances

File: examples/PlanarWalker/PlanarWalkerWithTorso.urdf (robot description, URDF)
Before this commit: robot KneedCompassGait, 13 links, 12 joints
Joints:
- joint torso_mass_weld: origin xyz=0 0 0 -> xyz=0 0 0.15

Commit message: added option for terminal mpc cost

File: examples/PlanarWalker/PlanarWalkerWithTorso.urdf (robot description, URDF)
Before this commit: robot KneedCompassGait, 13 links, 12 joints
Links:
- link left_lower_leg_mass: mass .125 -> 2
- link left_upper_leg_mass: mass 0.125 -> 5
- link right_lower_leg_mass: mass .125 -> 2
- link right_upper_leg_mass: mass .125 -> 5

Commit message: fixing gains and adding scripts for results testing

File: examples/PlanarWalker/PlanarWalkerWithTorso.urdf (robot description, URDF)
Before this commit: robot KneedCompassGait, 13 links, 12 joints
Links:
- link left_lower_leg_mass: mass 2 -> 1.5
- link left_upper_leg_mass: mass 5 -> 2.5
- link right_lower_leg_mass: mass 2 -> 1.5
- link right_upper_leg_mass: mass 5 -> 2.5
