Commit message: Merges from pinocchio branch.

File: examples/PlanarWalker/PlanarWalker.urdf (robot description, URDF)
Before this commit: robot KneedCompassGait, 12 links, 11 joints
Links:
- removed link base
- removed link base_x
- removed link base_xz
Joints:
- removed joint planar_roty
- removed joint planar_x
- removed joint planar_z
- joint hip_pin: limit (none) -> lower=-2 upper=2 effort=1e6 velocity=100
- joint left_knee_pin: limit effort=100 -> lower=-2 upper=2 effort=1e6 velocity=100
- joint right_knee_pin: limit effort=100 -> lower=-2 upper=2 effort=1e6 velocity=100

Commit message: Add inverse dynamics, also about 1/3 runtime as MBP.

File: examples/PlanarWalker/PlanarWalker.urdf (robot description, URDF)
Before this commit: robot KneedCompassGait, 9 links, 8 joints
Joints:
- joint hip_pin: type continuous -> revolute
- joint left_knee_pin: type continuous -> revolute

Commit message: Revert unwanted change from branch Pinnochio-merge

File: examples/PlanarWalker/PlanarWalker.urdf (robot description, URDF)
Before this commit: robot KneedCompassGait, 9 links, 8 joints
Links:
- added link base
- added link base_x
- added link base_xz
Joints:
- added joint planar_roty: type continuous, parent base_xz, child hip, axis 0 1 0
- added joint planar_x: type prismatic, parent base, child base_x, axis 1 0 0
- added joint planar_z: type prismatic, parent base_x, child base_xz, axis 0 0 1
- joint hip_pin: limit lower=-2 upper=2 effort=1e6 velocity=100 -> (none); type revolute -> continuous
- joint left_knee_pin: limit lower=-2 upper=2 effort=1e6 velocity=100 -> effort=100; type revolute -> continuous
- joint right_knee_pin: limit lower=-2 upper=2 effort=1e6 velocity=100 -> effort=100
