Commit message: Added stricter actuator limits

File: examples/five_link_biped/five_link_biped.urdf (robot description, URDF)
Before this commit: robot rabbit, 15 links, 14 joints
Joints:
- joint left_hip_pin: limit effort=300 -> effort=30
- joint left_knee_pin: limit effort=300 -> effort=30
- joint right_hip_pin: limit effort=300 -> effort=30
- joint right_knee_pin: limit effort=300 -> effort=30

Commit message: reading in actuator limits

File: examples/five_link_biped/five_link_biped.urdf (robot description, URDF)
Before this commit: robot rabbit, 15 links, 14 joints
Joints:
- joint left_hip_pin: limit effort=30 -> effort=35
- joint left_knee_pin: limit effort=30 -> effort=35
- joint right_hip_pin: limit effort=30 -> effort=35
- joint right_knee_pin: limit effort=30 -> effort=35
