Commit message: Added visualization for Spirit. run_spirit_vis.cc runs a zero trajectory used to see the spirit URDF in the visualizer with no optimization or step, will add animation of the legs. BUILD file was cobbled together to work and likely includes unecessary dependencies and the like, will clean up once I understand the build system and library a bit better.

File: examples/Spirit/xacros/spirit_drake.urdf.xacro (robot description, xacro)
@@ -67,4 +67,24 @@
 	<xacro:property name="jointSpeedLimit" value="30"/>
 	<xacro:property name="jointEffortLimit" value="40"/>
+	<xacro:property name="bodyColor" value="darkgray"/>
+	<xacro:property name="hipColor" value="copper"/>
+	<xacro:property name="upperLegColor" value="silver"/>
+	<xacro:property name="lowerLegColor" value="silver"/>
+	<xacro:property name="toeColor" value="black"/>
+	<material name="blue">
+      <color rgba="0 0 0.8 1"/>
+    </material>
+	<material name="black">
+      <color rgba="0.1 0.1 0.1 1"/>
+    </material>
+	<material name="darkgray">
+      <color rgba="0.25 0.25 0.25 1"/>
+    </material>
+	<material name="copper">
+      <color rgba="0.68 0.34 0.08 1"/>
+    </material>
+	<material name="silver">
+      <color rgba="0.68 0.68 0.68 1"/>
+    </material>
 	<!--
 	leg suffix="0" hipJointName="0" kneeJointName="1" abductionJointName="8"
@@ -80,5 +100,5 @@
 				<box size="${bodyLength} ${bodyWidth} ${bodyHeight}"/>
 			</geometry>
-			<material name="darkgray"/>
+			<material name="${bodyColor}"/>
 		</visual>
 		<inertial>
@@ -105,4 +125,5 @@
 					<cylinder length="${podLength}" radius="${podRadius}"/>
 				</geometry>
+				<material name="${hipColor}"/>
 			</visual>
 			<collision>
@@ -146,5 +167,5 @@
 					<box size="${upperLegLength} ${upperLegWidth} ${upperLegHeight}"/>
 				</geometry>
-				<material name="silver"/>
+				<material name="${upperLegColor}"/>
 			</visual>
 			<collision>
@@ -186,5 +207,5 @@
 					<cylinder length="${lowerLegLength}" radius="${lowerLegRadius}"/>
 				</geometry>
-				<material name="darkgray"/>
+				<material name="${lowerLegColor}"/>
 			</visual>
 			<collision>
@@ -233,5 +254,5 @@
 					<sphere radius="${toeRadius}"/>
 				</geometry>
-				<material name="darkgray"/>
+				<material name="${toeColor}"/>
 			</visual>
 			<collision>
