Commit message: Changed the xacro to include the joint_ to the joint names (previously 0-11) to more easily differentiate in printed debug statement and position_map dictionary calls. Added comments and animation to the run_spirit_vis.

File: examples/Spirit/spirit_drake.urdf (robot description, URDF)
Before this commit: robot spirit, 17 links, 16 joints
Joints:
- removed joint 0
- removed joint 1
- removed joint 10
- removed joint 11
- removed joint 2
- removed joint 3
- removed joint 4
- removed joint 5
- removed joint 6
- removed joint 7
- removed joint 8
- removed joint 9
- added joint joint_0: type revolute, parent hip0, child upper0, origin xyz=0.0 0.10098 0, axis 0 -1 0
- added joint joint_1: type revolute, parent upper0, child lower0, origin xyz=-0.206 0 0, axis 0 1 0
- added joint joint_10: type revolute, parent body, child hip2, origin xyz=0.2263 -0.07 0, axis 1 0 0
- added joint joint_11: type revolute, parent body, child hip3, origin xyz=-0.2263 -0.07 0, axis 1 0 0
- added joint joint_2: type revolute, parent hip1, child upper1, origin xyz=-0.0 0.10098 0, axis 0 -1 0
- added joint joint_3: type revolute, parent upper1, child lower1, origin xyz=-0.206 0 0, axis 0 1 0
- added joint joint_4: type revolute, parent hip2, child upper2, origin xyz=0.0 -0.10098 0, axis 0 -1 0
- added joint joint_5: type revolute, parent upper2, child lower2, origin xyz=-0.206 0 0, axis 0 1 0
- added joint joint_6: type revolute, parent hip3, child upper3, origin xyz=-0.0 -0.10098 0, axis 0 -1 0
- added joint joint_7: type revolute, parent upper3, child lower3, origin xyz=-0.206 0 0, axis 0 1 0
- added joint joint_8: type revolute, parent body, child hip0, origin xyz=0.2263 0.07 0, axis 1 0 0
- added joint joint_9: type revolute, parent body, child hip1, origin xyz=-0.2263 0.07 0, axis 1 0 0

File: examples/Spirit/xacros/spirit_drake.urdf.xacro (robot description, xacro)
@@ -141,10 +141,10 @@
 		</link>
 		<!-- Abduction joint. Joint names are: 8 9 10 11 -->
-		<joint name="${abductionJointName}" type="revolute">
+		<joint name="joint_${abductionJointName}" type="revolute">
 			<parent link="body"/>
 			<child link="hip${suffix}"/>
 			<axis xyz="1 0 0"/>
 			<origin xyz="${front * dx} ${left * dy} 0"/>
-			<limit effort="${abEffortLimit}" velocity="${abSpeedLimit}" lower="${-abKinLimit}" upper="${abKinLimit}"/>
+			<!-- <limit effort="${abEffortLimit}" velocity="${abSpeedLimit}" lower="${-abKinLimit}" upper="${abKinLimit}"/> -->
 			<dynamics damping="0.0" friction="0.0"/>
 		</joint>
@@ -152,5 +152,5 @@
 		<transmission name="transmission_${abductionJointName}">
     		<type>transmission_interface/SimpleTransmission</type>
-    		<joint name="${abductionJointName}">
+    		<joint name="joint_${abductionJointName}">
       			<!-- <hardwareInterface>hardware_interface/EffortJointInterface</hardwareInterface> -->
     		</joint>
@@ -181,10 +181,10 @@
 		</link>
 		<!-- Hip joint. (Motor to upper leg). Joint names are: 0 2 4 6 -->
-		<joint name="${hipJointName}" type="revolute">
+		<joint name="joint_${hipJointName}" type="revolute">
 			<parent link="hip${suffix}"/>
 			<child link="upper${suffix}"/>
 			<axis xyz="0 -1 0"/>
 			<origin xyz="${front * 0} ${left * abOffs} 0"/> <!--  rpy="0 -0.3 0" -->
-			<limit effort="${jointEffortLimit}" velocity="${jointSpeedLimit}" lower="${hipJointLowerLimit}" upper="${hipJointUpperLimit}"/>
+			<!-- <limit effort="${jointEffortLimit}" velocity="${jointSpeedLimit}" lower="${hipJointLowerLimit}" upper="${hipJointUpperLimit}"/> -->
 			<dynamics damping="0.0" friction="0.0"/>
 		</joint>
@@ -192,5 +192,5 @@
 		<transmission name="transmission_${hipJointName}">
     		<type>transmission_interface/SimpleTransmission</type>
-    		<joint name="${hipJointName}">
+    		<joint name="joint_${hipJointName}">
       			<!-- <hardwareInterface>hardware_interface/EffortJointInterface</hardwareInterface> -->
     		</joint>
@@ -221,10 +221,10 @@
 		</link>
 		<!-- Knee joint. Joint names are: 1 3 5 7 -->
-		<joint name="${kneeJointName}" type="revolute">
+		<joint name="joint_${kneeJointName}" type="revolute">
 			<parent link="upper${suffix}"/>
 			<child link="lower${suffix}"/>
 			<axis xyz="0 1 0"/>
 			<origin xyz="-${upperLegLength} 0 0"/> <!--rpy="0 0.5 0"-->
-			<limit effort="${jointEffortLimit}" velocity="${jointSpeedLimit}" lower="0" upper="${pi}"/>
+			<!-- <limit effort="${jointEffortLimit}" velocity="${jointSpeedLimit}" lower="0" upper="${pi}"/> -->
 			<dynamics damping="0.0" friction="0.0"/>
 		</joint>
@@ -232,5 +232,5 @@
 		<transmission name="transmission_${kneeJointName}">
     		<type>transmission_interface/SimpleTransmission</type>
-    		<joint name="${kneeJointName}">
+    		<joint name="joint_${kneeJointName}">
       			<!-- <hardwareInterface>hardware_interface/EffortJointInterface</hardwareInterface> -->
     		</joint>
