Commit message: fixed some bugs and wrote parameter learning script - still need to validate cube parameters against problem setup

File: examples/contact_parameter_learning/urdf/cube.urdf (robot description, URDF)
Before this commit: robot cube, 1 links, 0 joints
Links:
- link cube_base: geometry collision box size=0.1048 0.1048 0.1048; visual box size=0.1048 0.1048 0.1048
