Commit message: maybe working on force visualization

File: examples/simple_examples/urdf/finger_pen.urdf (robot description, URDF)
Before this commit: robot finger_pen, 9 links, 8 joints
Links:
- link bar1: geometry visual cylinder length=0.1 radius=0.051
- link bar2: geometry visual cylinder length=0.1 radius=0.051
- link bar3: geometry visual cylinder length=0.1 radius=0.051
