Commit message: Improvements to experiment setup
added flag for joint state channel in run_c3_ros_to_lcm and minor BAZEL changes

improved starting/stopping script, needs testing

moved boilerplate path finding code to function

minor changeS

slight change to q_init_finger, now represents height above table

script for updating urdf from parameters.yaml

integrate angular velocity for visualization

log parameters on c3 computer as well

File: examples/franka_trajectory_following/robot_properties_fingers/urdf/franka_box_template.urdf (robot description, URDF)
Before this commit: robot panda, 13 links, 12 joints
Links:
- link connection: geometry visual box size=0.3 0.3 TABLE_OFFSET
- link panda_link10: geometry collision sphere radius=FINGER_RADIUS; visual sphere radius=FINGER_RADIUS
Joints:
- joint connection_to_box: origin xyz=0 0 -0.0765 -> xyz=0 0 TABLE_ORIGIN
