Commit message: added squash ball EE to urdf

File: examples/franka_trajectory_following/robot_properties_fingers/urdf/franka_box.urdf (robot description, URDF)
Before this commit: robot panda, 10 links, 9 joints
Links:
- added link panda_link10; collision sphere radius=0.0198; visual sphere radius=0.0198
- added link panda_link9, mass 0.1340688; visual cylinder length=0.1016 radius=0.0127
- link panda_link8: mass None -> 0.0779312; geometry collision cylinder length=0.0096 radius=0.0315; visual cylinder length=0.0096 radius=0.0315
Joints:
- added joint panda_joint10: type fixed, parent panda_link9, child panda_link10, origin xyz=0 0 0.1016 rpy=0 0 0
- added joint panda_joint9: type fixed, parent panda_link8, child panda_link9, origin xyz=0 0 0.0096 rpy=0 0 0

Commit message: made necessary changes in other files to use new EE

File: examples/franka_trajectory_following/robot_properties_fingers/urdf/franka_box.urdf (robot description, URDF)
Before this commit: robot panda, 12 links, 11 joints
Links:
- link panda_link10: geometry collision sphere radius=0.0195; visual sphere radius=0.0195

Commit message: working with 0.01 radius and ok with 0.0195, lowered table

File: examples/franka_trajectory_following/robot_properties_fingers/urdf/franka_box.urdf (robot description, URDF)
Before this commit: robot panda, 12 links, 11 joints
Links:
- added link connection; visual box size=0.3 0.3 0.0301
Joints:
- removed joint box_to_base
- added joint base_to_connection: type fixed, parent panda_link0, child connection, origin xyz=0 0 0
- added joint connection_to_box: type fixed, parent connection, child box, origin xyz=0 0 -0.0801

Commit message: ran experiments: added json for EE, tweaked gains, tweaked target trajectory, fixed derivative issue in trajectory source code, updated procman, updated franka urdf to contain mass of ball

File: examples/franka_trajectory_following/robot_properties_fingers/urdf/franka_box.urdf (robot description, URDF)
Before this commit: robot panda, 13 links, 12 joints
Links:
- link panda_link10: mass None -> 0.057

Commit message: changed table offset

File: examples/franka_trajectory_following/robot_properties_fingers/urdf/franka_box.urdf (robot description, URDF)
Before this commit: robot panda, 13 links, 12 joints
Links:
- link connection: geometry visual box size=0.3 0.3 0.0235
Joints:
- joint connection_to_box: origin xyz=0 0 -0.0801 -> xyz=0 0 -0.0735

Commit message: sync with alp

File: examples/franka_trajectory_following/robot_properties_fingers/urdf/franka_box.urdf (robot description, URDF)
Before this commit: robot panda, 13 links, 12 joints
Links:
- link connection: geometry visual box size=0.3 0.3 0.0225
Joints:
- joint connection_to_box: origin xyz=0 0 -0.0735 -> xyz=0 0 -0.0725

Commit message: sync with alp

File: examples/franka_trajectory_following/robot_properties_fingers/urdf/franka_box.urdf (robot description, URDF)
Before this commit: robot panda, 13 links, 12 joints
Links:
- link connection: geometry visual box size=0.3 0.3 0.0245
Joints:
- joint connection_to_box: origin xyz=0 0 -0.0725 -> xyz=0 0 -0.0745

Commit message: sync with alp

File: examples/franka_trajectory_following/robot_properties_fingers/urdf/franka_box.urdf (robot description, URDF)
Before this commit: robot panda, 13 links, 12 joints
Links:
- link connection: geometry visual box size=0.3 0.3 0.0265
Joints:
- joint connection_to_box: origin xyz=0 0 -0.0745 -> xyz=0 0 -0.0765

Commit message: experiments from 08/12

File: examples/franka_trajectory_following/robot_properties_fingers/urdf/franka_box.urdf (robot description, URDF)
Before this commit: robot panda, 13 links, 12 joints
Links:
- link connection: geometry visual box size=0.3 0.3 0.0235
Joints:
- joint connection_to_box: origin xyz=0 0 -0.0765 -> xyz=0 0 -0.07350000000000001

Commit message: decent parameters experiment

File: examples/franka_trajectory_following/robot_properties_fingers/urdf/franka_box.urdf (robot description, URDF)
Before this commit: robot panda, 13 links, 12 joints
Links:
- link connection: geometry visual box size=0.3 0.3 0.0245
Joints:
- joint connection_to_box: origin xyz=0 0 -0.07350000000000001 -> xyz=0 0 -0.07450000000000001

Commit message: procman change

File: examples/franka_trajectory_following/robot_properties_fingers/urdf/franka_box.urdf (robot description, URDF)
Before this commit: robot panda, 13 links, 12 joints
Links:
- link connection: geometry visual box size=0.3 0.3 0.0235
Joints:
- joint connection_to_box: origin xyz=0 0 -0.07450000000000001 -> xyz=0 0 -0.07350000000000001

Commit message: syncing code from Franka computer

File: examples/franka_trajectory_following/robot_properties_fingers/urdf/franka_box.urdf (robot description, URDF)
Before this commit: robot panda, 13 links, 12 joints
Links:
- link connection: geometry visual box size=0.3 0.3 0.0242
Joints:
- joint connection_to_box: origin xyz=0 0 -0.07450000000000001 -> xyz=0 0 -0.0742

Commit message: first full circlesgit st! also my last day :D

File: examples/franka_trajectory_following/robot_properties_fingers/urdf/franka_box.urdf (robot description, URDF)
Before this commit: robot panda, 13 links, 12 joints
Links:
- link connection: geometry visual box size=0.3 0.3 0.0031
Joints:
- joint connection_to_box: origin xyz=0 0 -0.0742 -> xyz=0 0 -0.0531

Commit message: few hacks, might want to go back to previous commit

File: examples/franka_trajectory_following/robot_properties_fingers/urdf/franka_box.urdf (robot description, URDF)
Before this commit: robot panda, 13 links, 12 joints
Links:
- link connection: geometry visual box size=0.3 0.3 0.0245
Joints:
- joint connection_to_box: origin xyz=0 0 -0.0531 -> xyz=0 0 -0.07450000000000001

Commit message: fixed links to Franka meshes

File: examples/franka_trajectory_following/robot_properties_fingers/urdf/franka_box.urdf (robot description, URDF)
Before this commit: robot panda, 13 links, 12 joints
Links:
- link panda_link0: geometry collision sphere radius=0.06; collision sphere radius=0.06
- link panda_link1: geometry collision sphere radius=0.06; collision sphere radius=0.06
- link panda_link2: geometry collision sphere radius=0.06; collision sphere radius=0.06
- link panda_link3: geometry collision sphere radius=0.06; collision sphere radius=0.06
- link panda_link4: geometry collision sphere radius=0.05; collision sphere radius=0.055
- link panda_link5: geometry collision sphere radius=0.035; collision sphere radius=0.035
- link panda_link6: geometry collision sphere radius=0.05; collision sphere radius=0.06
- link panda_link7: geometry collision sphere radius=0.05; collision sphere radius=0.06

Commit message: merge more latest dairlib basic modules, robot_lcm_systems and multibody_utils, overload some function to stick to old usage for now, need more clean up in the future

File: examples/franka_trajectory_following/robot_properties_fingers/urdf/franka_box.urdf (robot description, URDF)
Before this commit: robot panda, 13 links, 12 joints
Links:
- link panda_link0: geometry collision sphere radius=0.06; collision sphere radius=0.06
- link panda_link1: geometry collision sphere radius=0.06; collision sphere radius=0.06
- link panda_link2: geometry collision sphere radius=0.06; collision sphere radius=0.06
- link panda_link3: geometry collision sphere radius=0.06; collision sphere radius=0.06
- link panda_link4: geometry collision sphere radius=0.05; collision sphere radius=0.055
- link panda_link5: geometry collision sphere radius=0.035; collision sphere radius=0.035
- link panda_link6: geometry collision sphere radius=0.05; collision sphere radius=0.06
- link panda_link7: geometry collision sphere radius=0.05; collision sphere radius=0.06
Joints:
- joint panda_joint10: origin xyz=0 0 0.0661 rpy=0 0 0 -> xyz=0 0 0.1016 rpy=0 0 0
- joint panda_joint8: origin xyz=0 0 0.1118 rpy=0 0 0 -> xyz=0 0 0.107 rpy=0 0 0
- joint panda_joint9: origin xyz=0 0 0.0556 rpy=0 0 0 -> xyz=0 0 0.0096 rpy=0 0 0
