Commit message: got prelim running trajectory

File: examples/impact_invariant_control/platform.urdf (robot description, URDF)
Before this commit: robot platform, 1 links, 0 joints
Links:
- link base: geometry collision box size=0.5 1.0 0.5; visual box size=0.5 1.0 0.5

Commit message: working on box jumping, need more conservative trajectories

File: examples/impact_invariant_control/platform.urdf (robot description, URDF)
Before this commit: robot platform, 1 links, 0 joints
Links:
- link base: geometry collision box size=0.5 1.0 0.2; visual box size=0.5 1.0 0.2

Commit message: need to debug box jumping controller

File: examples/impact_invariant_control/platform.urdf (robot description, URDF)
Before this commit: robot platform, 1 links, 0 joints
Links:
- link base: geometry collision box size=0.5 1.0 1.0; visual box size=0.5 1.0 1.0

Commit message: adding safety controllers

File: examples/impact_invariant_control/platform.urdf (robot description, URDF)
Before this commit: robot platform, 1 links, 0 joints
Links:
- link base: geometry collision box size=1.0 1.0 1.0; visual box size=1.0 1.0 1.0

Commit message: final sim visualization

File: examples/impact_invariant_control/platform.urdf (robot description, URDF)
Before this commit: robot platform, 1 links, 0 joints
Links:
- link base: geometry collision box size=1.0 1.0 0.5; visual box size=1.0 1.0 0.5
