Commit message: adding table in sim

File: examples/franka/urdf/franka_box.urdf (robot description, URDF)
Before this commit: robot panda, 13 links, 12 joints
Links:
- removed link box
- removed link connection
- removed link panda_link10
- removed link panda_link9
- link panda_link8: mass 0.0779312 -> 0.5; geometry collision box size=0.1 0.1 0.01; visual box size=0.1 0.1 0.01
Joints:
- removed joint base_to_connection
- removed joint connection_to_box
- removed joint panda_joint10
- removed joint panda_joint9

Commit message: moving table

File: examples/franka/urdf/franka_box.urdf (robot description, URDF)
Before this commit: robot panda, 9 links, 8 joints
Links:
- removed link panda_link8
- added link paddle, mass 0.5; collision box size=0.2 0.2 0.01; visual box size=0.2 0.2 0.01
Joints:
- removed joint panda_joint8
- added joint fixed_paddle: type fixed, parent panda_link7, child paddle, origin xyz=0 0 0.107 rpy=0 0 0
