Commit message: adding feed forward term

File: examples/franka/urdf/franka_no_collision.urdf (robot description, URDF)
Before this commit: robot panda, 9 links, 8 joints
Links:
- link paddle: geometry collision box size=0.5 0.5 0.02; visual box size=0.5 0.5 0.02

File: examples/franka/urdf/plate_end_effector_translation.urdf (robot description, URDF)
Before this commit: robot plate, 4 links, 3 joints
Links:
- link plate: geometry collision sphere radius=0.001; collision sphere radius=0.001
