Commit message: using better organized vector

File: examples/franka/urdf/plate_end_effector_floating.urdf (robot description, URDF)
Before this commit: robot plate, 4 links, 3 joints
Links:
- added link plate_rx
- added link plate_ry
- added link plate_rz
Joints:
- added joint plate_rx: type revolute, parent plate_rx, child plate_ry, axis 1 0 0
- added joint plate_ry: type revolute, parent plate_ry, child plate_rz, axis 0 1 0
- added joint plate_rz: type revolute, parent plate_rz, child plate, axis 0 0 1
- joint plate_z: child plate -> plate_rx

Commit message: working on orientatino

File: examples/franka/urdf/plate_end_effector_floating.urdf (robot description, URDF)
Before this commit: robot plate, 7 links, 6 joints
Links:
- link plate: mass 2 -> 0.5; geometry collision sphere radius=0.001; collision sphere radius=0.001

Commit message: checking parameters and urdfs

File: examples/franka/urdf/plate_end_effector_floating.urdf (robot description, URDF)
Before this commit: robot plate, 7 links, 6 joints
Links:
- link plate: mass 0.5 -> 2.0; geometry collision sphere radius=0.001; collision sphere radius=0.001
