Commit message: compilation settings

File: examples/franka/urdf/franka.urdf (robot description, URDF)
Before this commit: robot panda, 9 links, 8 joints
Links:
- link paddle: geometry collision box size=0.2 0.2 0.01; visual box size=0.2 0.2 0.01

Commit message: small debugging, also changing end effector width to avoid conflicting collision geometries

File: examples/franka/urdf/franka.urdf (robot description, URDF)
Before this commit: robot panda, 9 links, 8 joints
Links:
- link paddle: geometry collision box size=0.2 0.2 0.02; visual box size=0.2 0.2 0.02

Commit message: small trajectory tweaks

File: examples/franka/urdf/franka.urdf (robot description, URDF)
Before this commit: robot panda, 9 links, 8 joints
Links:
- link paddle: geometry collision box size=0.5 0.5 0.02; visual box size=0.5 0.5 0.02

Commit message: added orientation

File: examples/franka/urdf/franka.urdf (robot description, URDF)
Before this commit: robot panda, 9 links, 8 joints
Links:
- link paddle: geometry collision box size=0.2 0.2 0.02; visual box size=0.2 0.2 0.02

File: examples/franka/urdf/franka_no_collision.urdf (robot description, URDF)
Before this commit: robot panda, 9 links, 8 joints
Links:
- link paddle: geometry collision box size=0.2 0.2 0.02; visual box size=0.2 0.2 0.02

Commit message: drake master changes

File: examples/franka/urdf/franka.urdf (robot description, URDF)
Before this commit: robot panda, 9 links, 8 joints
Links:
- link panda_link0: geometry collision sphere radius=0.06; collision sphere radius=0.06
- link panda_link1: geometry collision sphere radius=0.06; collision sphere radius=0.06
- link panda_link2: geometry collision sphere radius=0.06; collision sphere radius=0.06
- link panda_link3: geometry collision sphere radius=0.06; collision sphere radius=0.06
- link panda_link4: geometry collision sphere radius=0.05; collision sphere radius=0.055
- link panda_link5: geometry collision sphere radius=0.035; collision sphere radius=0.035
- link panda_link6: geometry collision sphere radius=0.05; collision sphere radius=0.06
- link panda_link7: geometry collision sphere radius=0.05; collision sphere radius=0.06

File: examples/franka/urdf/franka_no_collision.urdf (robot description, URDF)
Before this commit: robot panda, 9 links, 8 joints
Links:
- link panda_link0: geometry visual mesh filename=package://drake_models/franka_description/meshes/visual/lin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
- link panda_link1: geometry visual mesh filename=package://drake_models/franka_description/meshes/visual/lin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
- link panda_link2: geometry visual mesh filename=package://drake_models/franka_description/meshes/visual/lin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
- link panda_link3: geometry visual mesh filename=package://drake_models/franka_description/meshes/visual/lin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
- link panda_link4: geometry visual mesh filename=package://drake_models/franka_description/meshes/visual/lin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
- link panda_link5: geometry visual mesh filename=package://drake_models/franka_description/meshes/visual/lin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
- link panda_link6: geometry visual mesh filename=package://drake_models/franka_description/meshes/visual/lin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
- link panda_link7: geometry visual mesh filename=package://drake_models/franka_description/meshes/visual/lin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

Commit message: need to fix jitter

File: examples/franka/urdf/franka.urdf (robot description, URDF)
Before this commit: robot panda, 9 links, 8 joints
Links:
- link paddle: geometry collision box size=0.5 0.5 0.02; visual box size=0.5 0.5 0.02

File: examples/franka/urdf/franka_no_collision.urdf (robot description, URDF)
Before this commit: robot panda, 9 links, 8 joints
Links:
- link paddle: geometry collision box size=0.5 0.5 0.02; visual box size=0.5 0.5 0.02

Commit message: plotting target position from c3 plan

File: examples/franka/urdf/franka.urdf (robot description, URDF)
Before this commit: robot panda, 9 links, 8 joints
Links:
- link paddle: mass 0.5 -> 1.0

Commit message: updates to 22.04

File: examples/franka/urdf/franka.urdf (robot description, URDF)
Before this commit: robot panda, 9 links, 8 joints
Links:
- link paddle: geometry collision box size=0.4 0.4 0.02; visual box size=0.4 0.4 0.02
- link panda_link0: geometry collision sphere radius=0.06; collision sphere radius=0.06
- link panda_link1: geometry collision sphere radius=0.06; collision sphere radius=0.06
- link panda_link2: geometry collision sphere radius=0.06; collision sphere radius=0.06
- link panda_link3: geometry collision sphere radius=0.06; collision sphere radius=0.06
- link panda_link4: geometry collision sphere radius=0.05; collision sphere radius=0.055
- link panda_link5: geometry collision sphere radius=0.035; collision sphere radius=0.035
- link panda_link6: geometry collision sphere radius=0.05; collision sphere radius=0.06
- link panda_link7: geometry collision sphere radius=0.05; collision sphere radius=0.06

File: examples/franka/urdf/franka_no_collision.urdf (robot description, URDF)
Before this commit: robot panda, 9 links, 8 joints
Links:
- link paddle: geometry collision box size=0.4 0.4 0.02; visual box size=0.4 0.4 0.02
- link panda_link0: geometry visual mesh filename=package://drake_models/franka_description/meshes/visual/lin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
- link panda_link1: geometry visual mesh filename=package://drake_models/franka_description/meshes/visual/lin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
- link panda_link2: geometry visual mesh filename=package://drake_models/franka_description/meshes/visual/lin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
- link panda_link3: geometry visual mesh filename=package://drake_models/franka_description/meshes/visual/lin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
- link panda_link4: geometry visual mesh filename=package://drake_models/franka_description/meshes/visual/lin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
- link panda_link5: geometry visual mesh filename=package://drake_models/franka_description/meshes/visual/lin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
- link panda_link6: geometry visual mesh filename=package://drake_models/franka_description/meshes/visual/lin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
- link panda_link7: geometry visual mesh filename=package://drake_models/franka_description/meshes/visual/lin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

File: examples/franka/urdf/plate_end_effector_floating.urdf (robot description, URDF)
Before this commit: robot plate, 7 links, 6 joints
Links:
- link plate: mass 2.0 -> 2

File: examples/franka/urdf/plate_end_effector_translation.urdf (robot description, URDF)
Before this commit: robot plate, 4 links, 3 joints
Links:
- link plate: mass 2.0 -> 2
