Commit message: still investigating contact model

File: examples/franka/urdf/left_support_point_contact.urdf (robot description, URDF)
Before this commit: robot left_support, 1 links, 0 joints
Links:
- link support: geometry collision sphere radius=0.001; collision sphere radius=0.001

Commit message: using point contact and box model now

File: examples/franka/urdf/left_support_point_contact.urdf (robot description, URDF)
Before this commit: robot left_support, 1 links, 0 joints
Links:
- link support: geometry collision box size=0.4 0.02 0.0481; collision sphere radius=0.001

Commit message: features implemented, need to tune with plots'

File: examples/franka/urdf/left_support_point_contact.urdf (robot description, URDF)
Before this commit: robot left_support, 1 links, 0 joints
Links:
- link support: geometry collision box size=0.1 0.02 0.05; collision sphere radius=0.001
