Commit message: double chekcing urdfs

File: examples/franka/urdf/plate_end_effector_translation.urdf (robot description, URDF)
Before this commit: robot plate, 4 links, 3 joints
Links:
- link plate: geometry collision sphere radius=0.01; collision sphere radius=0.01

Commit message: removing tables from franka examples

File: examples/franka/urdf/plate_end_effector_translation.urdf (robot description, URDF)
Before this commit: robot plate, 4 links, 3 joints
Links:
- link plate: mass 2 -> 1; geometry collision sphere radius=0.001; collision sphere radius=0.001

Commit message: updating end effector urdf from physical model

File: examples/franka/urdf/plate_end_effector_translation.urdf (robot description, URDF)
Before this commit: robot plate, 4 links, 3 joints
Links:
- link plate: mass 1 -> 0.37; geometry collision sphere radius=0.001; collision sphere radius=0.001

Commit message: changing w support demo

File: examples/franka/urdf/plate_end_effector_translation.urdf (robot description, URDF)
Before this commit: robot plate, 4 links, 3 joints
Links:
- link plate: geometry collision sphere radius=0.001; collision sphere radius=0.001
