Commit message: separating scene to separate yaml

File: examples/franka/urdf/support_point_contact.urdf (robot description, URDF)
Before this commit: robot left_support, 1 links, 0 joints
Links:
- removed link support
- added link base, mass 2; collision sphere radius=0.001; collision sphere radius=0.001
