Commit message: Added visualization for optimistic state prediction with solved with relaxed constraints. Increased thickness of table. Made table & jack translucent for better visualization.

File: examples/cube_franka/robot_properties_fingers/urdf/franka_box.urdf (robot description, URDF)
Before this commit: robot panda, 13 links, 12 joints
Links:
- link box: geometry collision box size=5 5 1.1; visual box size=5 5 1.1
Joints:
- joint connection_to_box: origin xyz=0 0 -0.07450000000000001 -> xyz=0 0 -0.57450000000000001

Commit message: Make jack and table opaque

File: examples/cube_franka/robot_properties_fingers/urdf/franka_box.urdf (robot description, URDF)
Before this commit: robot panda, 13 links, 12 joints
Links:
- link box: geometry collision box size=5 5 0.1; visual box size=5 5 0.1
Joints:
- joint connection_to_box: origin xyz=0 0 -0.57450000000000001 -> xyz=0 0 -0.07450000000000001

Commit message: Added changes for flask UI to display each visualization attribute as a checkbox.

File: examples/cube_franka/robot_properties_fingers/urdf/franka_box.urdf (robot description, URDF)
Before this commit: robot panda, 13 links, 12 joints
Links:
- link panda_link0: geometry collision sphere radius=0.06; collision sphere radius=0.06
- link panda_link1: geometry collision sphere radius=0.06; collision sphere radius=0.06
- link panda_link2: geometry collision sphere radius=0.06; collision sphere radius=0.06
- link panda_link3: geometry collision sphere radius=0.06; collision sphere radius=0.06
- link panda_link4: geometry collision sphere radius=0.05; collision sphere radius=0.055
- link panda_link5: geometry collision sphere radius=0.035; collision sphere radius=0.035
- link panda_link6: geometry collision sphere radius=0.05; collision sphere radius=0.06
- link panda_link7: geometry collision sphere radius=0.05; collision sphere radius=0.06

File: examples/cube_franka/robot_properties_fingers/urdf/franka_box_template.urdf (robot description, URDF)
Before this commit: robot panda, 13 links, 12 joints
Links:
- link panda_link0: geometry collision sphere radius=0.06; collision sphere radius=0.06
- link panda_link1: geometry collision sphere radius=0.06; collision sphere radius=0.06
- link panda_link2: geometry collision sphere radius=0.06; collision sphere radius=0.06
- link panda_link3: geometry collision sphere radius=0.06; collision sphere radius=0.06
- link panda_link4: geometry collision sphere radius=0.05; collision sphere radius=0.055
- link panda_link5: geometry collision sphere radius=0.035; collision sphere radius=0.035
- link panda_link6: geometry collision sphere radius=0.05; collision sphere radius=0.06
- link panda_link7: geometry collision sphere radius=0.05; collision sphere radius=0.06

File: examples/franka/robot_properties_fingers/urdf/franka_box.urdf (robot description, URDF)
Before this commit: robot panda, 10 links, 9 joints
Links:
- link panda_link0: geometry collision sphere radius=0.06; collision sphere radius=0.06
- link panda_link1: geometry collision sphere radius=0.06; collision sphere radius=0.06
- link panda_link2: geometry collision sphere radius=0.06; collision sphere radius=0.06
- link panda_link3: geometry collision sphere radius=0.06; collision sphere radius=0.06
- link panda_link4: geometry collision sphere radius=0.05; collision sphere radius=0.055
- link panda_link5: geometry collision sphere radius=0.035; collision sphere radius=0.035
- link panda_link6: geometry collision sphere radius=0.05; collision sphere radius=0.06
- link panda_link7: geometry collision sphere radius=0.05; collision sphere radius=0.06
