Commit message: - Removed mode_selector system - Moved preprocessing step into controller for continuous resolution of contact points - Fixed end effector frame weld to have it be oriented downward - Removed most scene indexing - Fixed connections in controller - Added some visualization systems - Fixed sizes of friction vector/g_x/g_lambda etc - Removed unused yaml files - Fixed memory errors relating to undefined sizes in the LCS matrices. - Fixed definitions of Update traj functions to include position/orientation/force trajectories. - Added clear trajectories method to LcmTrajectory class. - Fixed solve time filtering snippet - Included diagrams for reference - Currently fixing TrackingTrajGenerator definition to look for newly added trajectories along with unique naming of visualization systems.

File: examples/jacktoy/urdf/end_effector_full.urdf (robot description, URDF)
Before this commit: robot end_effector_full, 3 links, 2 joints
Joints:
- joint fix_link_base: origin xyz=0 0 0.0096 rpy=0 0 0 -> xyz=0 0 -0.0096 rpy=0 0 0
- joint fix_tip_link: origin xyz=0 0 0.1016 rpy=0 0 0 -> xyz=0 0 -0.1016 rpy=0 0 0

Commit message: Make origin of end effector tip match center of sphere geometry

File: examples/jacktoy/urdf/end_effector_full.urdf (robot description, URDF)
Before this commit: robot end_effector_full, 3 links, 2 joints
Joints:
- joint fix_tip_link: origin xyz=0 0 -0.1016 rpy=0 0 0 -> xyz=0 0 -0.1169 rpy=0 0 0
