Commit message: - Fixed visualization for lcs state. - added a transparency parameter to multipose visualizer. - Removed end_effector_thickness from params file.

File: examples/jacktoy/urdf/c3_mode_visualization.urdf (robot description, URDF)
Before this commit: robot sample_sphere, 1 links, 0 joints
Links:
- link sample_sphere: geometry visual sphere radius=0.0198
