Commit message: -Fixed urdf and model offsets. -renamed frames in yamls -Tuned safe parameters along with workspace constraints -Made ee_min_z_height a param for C3

File: examples/jacktoy/urdf/platform.urdf (robot description, URDF)
Before this commit: robot platform, 1 links, 0 joints
Links:
- link platform: geometry visual box size=0.3 0.3 0.029

Commit message: Make robot platform in simulation more closely match hardware

File: examples/jacktoy/urdf/platform.urdf (robot description, URDF)
Before this commit: robot platform, 1 links, 0 joints
Links:
- link platform: geometry collision box size=0.3 0.6 0.029; visual box size=0.3 0.6 0.029
