Commit message: solve the not ideal urdf definition problem, now the end-effector frame is directly alligned with sphere center

File: examples/franka_ball_rolling/robot_properties_fingers/urdf/end_effector_full.urdf (robot description, URDF)
Before this commit: robot end_effector_full, 3 links, 2 joints
Joints:
- joint fix_link_base: origin xyz=0 0 0.0096 rpy=0 0 0 -> xyz=0 0 0.0556 rpy=0 0 0
- joint fix_tip_link: origin xyz=0 0 0.1016 rpy=0 0 0 -> xyz=0 0 0.0661 rpy=0 0 0

File: examples/franka_trajectory_following/robot_properties_fingers/urdf/franka_box.urdf (robot description, URDF)
Before this commit: robot panda, 13 links, 12 joints
Joints:
- joint panda_joint10: origin xyz=0 0 0.1016 rpy=0 0 0 -> xyz=0 0 0.0661 rpy=0 0 0
- joint panda_joint8: origin xyz=0 0 0.107 rpy=0 0 0 -> xyz=0 0 0.1118 rpy=0 0 0
- joint panda_joint9: origin xyz=0 0 0.0096 rpy=0 0 0 -> xyz=0 0 0.0556 rpy=0 0 0
