Commit message: Bug fix in ROS2 integration

File: examples/trifinger/robot_properties_fingers/urdf/edu/trifingeredu.urdf (robot description, URDF)
Before this commit: robot trifingeredu, 17 links, 16 joints
Links:
- link finger_base_link_0: geometry collision mesh filename=../meshes/edu/base_back.obj scale=1 1 1; collision mesh filename=../meshes/edu/base_front.obj scale=1 1 1
- link finger_base_link_120: geometry collision mesh filename=../meshes/edu/base_back.obj scale=1 1 1; collision mesh filename=../meshes/edu/base_front.obj scale=1 1 1
- link finger_base_link_240: geometry collision mesh filename=../meshes/edu/base_back.obj scale=1 1 1; collision mesh filename=../meshes/edu/base_front.obj scale=1 1 1
- link finger_lower_link_0: geometry collision mesh filename=../meshes/edu/lower_link.obj scale=1 1 1; visual mesh filename=../meshes/edu/lower_link.obj scale=1 1 1
- link finger_lower_link_120: geometry collision mesh filename=../meshes/edu/lower_link.obj scale=1 1 1; visual mesh filename=../meshes/edu/lower_link.obj scale=1 1 1
- link finger_lower_link_240: geometry collision mesh filename=../meshes/edu/lower_link.obj scale=1 1 1; visual mesh filename=../meshes/edu/lower_link.obj scale=1 1 1
- link finger_middle_link_0: geometry collision mesh filename=../meshes/edu/middle_link.obj scale=1 1 1; visual mesh filename=../meshes/edu/middle_link.obj scale=1 1 1
- link finger_middle_link_120: geometry collision mesh filename=../meshes/edu/middle_link.obj scale=1 1 1; visual mesh filename=../meshes/edu/middle_link.obj scale=1 1 1
- link finger_middle_link_240: geometry collision mesh filename=../meshes/edu/middle_link.obj scale=1 1 1; visual mesh filename=../meshes/edu/middle_link.obj scale=1 1 1
- link finger_upper_link_0: geometry collision mesh filename=../meshes/edu/upper_link.obj scale=1 1 1; visual mesh filename=../meshes/edu/upper_link.obj scale=1 1 1
- link finger_upper_link_120: geometry collision mesh filename=../meshes/edu/upper_link.obj scale=1 1 1; visual mesh filename=../meshes/edu/upper_link.obj scale=1 1 1
- link finger_upper_link_240: geometry collision mesh filename=../meshes/edu/upper_link.obj scale=1 1 1; visual mesh filename=../meshes/edu/upper_link.obj scale=1 1 1

Commit message: Change link mass values in the trifinger urdf

File: examples/trifinger/robot_properties_fingers/urdf/edu/trifingeredu.urdf (robot description, URDF)
Before this commit: robot trifingeredu, 17 links, 16 joints
Links:
- link finger_lower_link_0: mass 0.03070 -> 0.035
- link finger_lower_link_120: mass 0.03070 -> 0.035
- link finger_lower_link_240: mass 0.03070 -> 0.035
- link finger_middle_link_0: mass 0.14854 -> 0.16
- link finger_middle_link_120: mass 0.14854 -> 0.16
- link finger_middle_link_240: mass 0.14854 -> 0.16
- link finger_upper_link_0: mass 0.14854 -> 0.157
- link finger_upper_link_120: mass 0.14854 -> 0.157
- link finger_upper_link_240: mass 0.14854 -> 0.157
Joints:
- joint base_to_finger_0: origin xyz=-0.0455 0.0 0 rpy=0 0 0 -> xyz=-0.0395 0.0 0 rpy=0 0 0
- joint base_to_finger_120: origin xyz=0.02274999999999999 0.03940415587219196 0 rpy=0 0 -2.0943951023931953 -> xyz=0.01975 0.034208 0 rpy=0 0 -2.0943951023931953
- joint base_to_finger_240: origin xyz=0.02275000000000002 -0.03940415587219195 0 rpy=0 0 -4.1887902047863905 -> xyz=0.01975 -0.034208 0 rpy=0 0 -4.1887902047863905
- joint base_to_trifinger_base_joint: origin xyz=0 0 0.283 rpy=0 0 -1.5707963267948966 -> xyz=0 0 0.282 rpy=0 0 -1.5707963267948966

Commit message: Fix limits of joint torques in trifinger urdf

File: examples/trifinger/robot_properties_fingers/urdf/edu/trifingeredu.urdf (robot description, URDF)
Before this commit: robot trifingeredu, 17 links, 16 joints
Joints:
- joint finger_base_to_upper_joint_0: limit lower=-1.5707963267948966 upper=1.5707963267948966 effort=1000 velocity=1000 -> lower=-1.5707963267948966 upper=1.5707963267948966 effort=0.36 velocity=20
- joint finger_base_to_upper_joint_120: limit lower=-1.5707963267948966 upper=1.5707963267948966 effort=1000 velocity=1000 -> lower=-1.5707963267948966 upper=1.5707963267948966 effort=0.36 velocity=20
- joint finger_base_to_upper_joint_240: limit lower=-1.5707963267948966 upper=1.5707963267948966 effort=1000 velocity=1000 -> lower=-1.5707963267948966 upper=1.5707963267948966 effort=0.36 velocity=20
- joint finger_middle_to_lower_joint_0: limit lower=-3.141592653589793 upper=3.141592653589793 effort=1000 velocity=1000 -> lower=-3.141592653589793 upper=3.141592653589793 effort=0.36 velocity=20
- joint finger_middle_to_lower_joint_120: limit lower=-3.141592653589793 upper=3.141592653589793 effort=1000 velocity=1000 -> lower=-3.141592653589793 upper=3.141592653589793 effort=0.36 velocity=20
- joint finger_middle_to_lower_joint_240: limit lower=-3.141592653589793 upper=3.141592653589793 effort=1000 velocity=1000 -> lower=-3.141592653589793 upper=3.141592653589793 effort=0.36 velocity=20
- joint finger_upper_to_middle_joint_0: limit lower=-1.5707963267948966 upper=1.5707963267948966 effort=1000 velocity=1000 -> lower=-1.5707963267948966 upper=1.5707963267948966 effort=0.36 velocity=20
- joint finger_upper_to_middle_joint_120: limit lower=-1.5707963267948966 upper=1.5707963267948966 effort=1000 velocity=1000 -> lower=-1.5707963267948966 upper=1.5707963267948966 effort=0.36 velocity=20
- joint finger_upper_to_middle_joint_240: limit lower=-1.5707963267948966 upper=1.5707963267948966 effort=1000 velocity=1000 -> lower=-1.5707963267948966 upper=1.5707963267948966 effort=0.36 velocity=20

Commit message: updated URDF

File: examples/trifinger/robot_properties_fingers/urdf/edu/trifingeredu.urdf (robot description, URDF)
Before this commit: robot trifingeredu, 17 links, 16 joints
Links:
- removed link finger_tip_link_0
- removed link finger_tip_link_120
- added link densetact_0, mass 0.035; collision sphere radius=0.01575; visual mesh filename=../meshes/edu/finger_tip_dt2.obj scale=0.001 0.001 0.001
- added link densetact_120, mass 0.035; collision sphere radius=0.01575; visual mesh filename=../meshes/edu/finger_tip_dt1.obj scale=0.001 0.001 0.001
- added link optical_center_0
- added link optical_center_120
- link finger_lower_link_0: geometry collision mesh filename=../meshes/edu/link_mount_dt2.obj scale=0.001 0.001 0.001; visual mesh filename=../meshes/edu/link_mount_dt2.obj scale=0.001 0.001 0.001
- link finger_lower_link_120: geometry collision mesh filename=../meshes/edu/link_mount_dt1.obj scale=0.001 0.001 0.001; visual mesh filename=../meshes/edu/link_mount_dt1.obj scale=0.001 0.001 0.001
Joints:
- removed joint finger_lower_to_tip_joint_0
- removed joint finger_lower_to_tip_joint_120
- added joint densetact_0_to_optical_center: type fixed, parent densetact_0, child optical_center_0, origin xyz=0 0 0.00360 rpy=0 0 0
- added joint densetact_120_to_optical_center: type fixed, parent densetact_120, child optical_center_120, origin xyz=0 0 0.00360 rpy=0 0 0
- added joint mount_to_densetact_0: type fixed, parent finger_lower_link_0, child densetact_0, origin xyz=0 -0.008 -0.14985 rpy=0 0 0
- added joint mount_to_densetact_120: type fixed, parent finger_lower_link_120, child densetact_120, origin xyz=0 -0.008 -0.151974 rpy=0 0 0

Commit message: contact info from densetact

File: examples/trifinger/robot_properties_fingers/urdf/edu/trifingeredu.urdf (robot description, URDF)
Before this commit: robot trifingeredu, 19 links, 18 joints
Links:
- link finger_base_link_0: geometry collision mesh filename=../meshes/edu/base_back.obj scale=1 1 1; collision mesh filename=../meshes/edu/base_side_left.obj scale=1 1 1
