Commit message: Added DenseTact visualization to trifinger visualizer

File: examples/trifinger/robot_properties_fingers/urdf/edu/dualfingeredu.urdf (robot description, URDF)
Before this commit: robot trifingeredu, 19 links, 18 joints
Links:
- added link densetact_0_vis; visual mesh filename=../meshes/edu/finger_tip_dt1.obj scale=0.001 0.001 0.001
- added link densetact_120_vis; visual mesh filename=../meshes/edu/finger_tip_dt2.obj scale=0.001 0.001 0.001
- link densetact_0: geometry collision sphere radius=0.01575; visual sphere radius=0.01575
- link densetact_120: geometry collision sphere radius=0.01575; visual sphere radius=0.01575
- link finger_lower_link_0: geometry collision mesh filename=../meshes/edu/link_mount_dt1.obj scale=0.001 0.001 0.001; visual mesh filename=../meshes/edu/link_mount_dt1.obj scale=0.001 0.001 0.001
- link finger_lower_link_120: geometry collision mesh filename=../meshes/edu/link_mount_dt2.obj scale=0.001 0.001 0.001; visual mesh filename=../meshes/edu/link_mount_dt2.obj scale=0.001 0.001 0.001
Joints:
- added joint densetact_0_to_vis: type fixed, parent densetact_0, child densetact_0_vis, origin xyz=0 0 0 rpy=0 0 0
- added joint densetact_120_to_vis: type fixed, parent densetact_120, child densetact_120_vis, origin xyz=0 0 0 rpy=0 0 0
- joint mount_to_densetact_0: origin xyz=0 -0.008 -0.14985 rpy=0 0 0 -> xyz=-0.005 -0.01 -0.140974 rpy=0 0 0
- joint mount_to_densetact_120: origin xyz=0 -0.008 -0.151974 rpy=0 0 0 -> xyz=0 -0.008 -0.14785 rpy=0 0 0

Commit message: Add all dice meshes to visualizer

File: examples/trifinger/robot_properties_fingers/urdf/edu/dualfingeredu.urdf (robot description, URDF)
Before this commit: robot trifingeredu, 21 links, 20 joints
Links:
- removed link densetact_0_vis
- removed link densetact_120_vis
- link densetact_0: geometry visual mesh filename=../meshes/edu/finger_tip_dt1.obj scale=0.001 0.001 0.001
- link densetact_120: geometry visual mesh filename=../meshes/edu/finger_tip_dt2.obj scale=0.001 0.001 0.001
- link optical_center_0: geometry collision sphere radius=0.01575; visual sphere radius=0.01575
- link optical_center_120: geometry collision sphere radius=0.01575; visual sphere radius=0.01575
Joints:
- removed joint densetact_0_to_vis
- removed joint densetact_120_to_vis
- joint densetact_0_to_optical_center: origin xyz=0 0 0.00360 rpy=0 0 0 -> xyz=0 0 0 rpy=0 3.14159 1.57079
- joint densetact_120_to_optical_center: origin xyz=0 0 0.00360 rpy=0 0 0 -> xyz=0 0 0 rpy=0 3.14159 1.57079

Commit message: Hand-calibration of distal link and densetact optical center

File: examples/trifinger/robot_properties_fingers/urdf/edu/dualfingeredu.urdf (robot description, URDF)
Before this commit: robot trifingeredu, 19 links, 18 joints
Joints:
- joint mount_to_densetact_0: origin xyz=-0.005 -0.01 -0.140974 rpy=0 0 0 -> xyz=-0.005 -0.01 -0.142974 rpy=0 0 0
- joint mount_to_densetact_120: origin xyz=0 -0.008 -0.14785 rpy=0 0 0 -> xyz=0 -0.008 -0.14485 rpy=0 0 0
