Commit message: Working as of May 11

File: examples/trifinger/robot_properties_fingers/urdf/edu/dualfingeredu_original.urdf (robot description, URDF)
Before this commit: robot trifingeredu, 19 links, 18 joints
Links:
- removed link densetact_0
- removed link densetact_120
- removed link optical_center_0
- removed link optical_center_120
- added link finger_tip_link_0, mass 0.01
- added link finger_tip_link_120, mass 0.01
- link finger_base_link_240: mass 1 -> None; geometry 
- link finger_lower_link_0: geometry collision mesh filename=../meshes/edu/lower_link.obj scale=1 1 1; visual mesh filename=../meshes/edu/lower_link.obj scale=1 1 1
- link finger_lower_link_120: geometry collision mesh filename=../meshes/edu/lower_link.obj scale=1 1 1; visual mesh filename=../meshes/edu/lower_link.obj scale=1 1 1
- link finger_lower_link_240: mass 0.035 -> None; geometry 
- link finger_middle_link_240: mass 0.16 -> None; geometry 
- link finger_tip_link_240: mass 0.01 -> None
- link finger_upper_link_240: geometry 
Joints:
- removed joint densetact_0_to_optical_center
- removed joint densetact_120_to_optical_center
- removed joint mount_to_densetact_0
- removed joint mount_to_densetact_120
- added joint finger_lower_to_tip_joint_0: type fixed, parent finger_lower_link_0, child finger_tip_link_0, origin xyz=0 -0.008 -0.16
- added joint finger_lower_to_tip_joint_120: type fixed, parent finger_lower_link_120, child finger_tip_link_120, origin xyz=0 -0.008 -0.16
- joint base_to_finger_0: origin xyz=-0.004 -0.043 0 rpy=0 0 1.570796 -> xyz=0 -0.045 0 rpy=0 0 1.570796
- joint base_to_finger_120: origin xyz=0.005 0.045 0 rpy=0 0 -1.570796 -> xyz=0 0.045 -0.002 rpy=0 0 -1.570796
- joint base_to_finger_240: origin xyz=-0.98025 -0.034208 0 rpy=0 0 -4.1887902047863905 -> xyz=0.01975 -0.034208 0 rpy=0 0 -4.1887902047863905
- joint finger_middle_to_lower_joint_0: origin xyz=0.005 -0.03745 -0.16 rpy=0 0 0 -> xyz=0 -0.03745 -0.16 rpy=0 0 0
