Commit message: T changed to 16x4x4cm. Smaller end effector and corresponding visualization models.

File: examples/push_T/urdf/c3_mode_visualization.urdf (robot description, URDF)
Before this commit: robot sample_sphere, 1 links, 0 joints
Links:
- link sample_sphere: geometry visual sphere radius=0.0146

File: examples/push_T/urdf/sample_locations.urdf (robot description, URDF)
Before this commit: robot sample_sphere, 1 links, 0 joints
Links:
- link sample_sphere: geometry visual sphere radius=0.0145

Commit message: Updated end-effector to match the hardware. Added tuned params from log 112 Mar 14th.

File: examples/push_T/urdf/c3_mode_visualization.urdf (robot description, URDF)
Before this commit: robot sample_sphere, 1 links, 0 joints
Links:
- link sample_sphere: geometry visual sphere radius=0.0196

File: examples/push_T/urdf/ee_best_traj_visualization_model.urdf (robot description, URDF)
Before this commit: robot end_effector_simple, 1 links, 0 joints
Links:
- link end_effector_simple: geometry visual sphere radius=0.0195

File: examples/push_T/urdf/ee_curr_traj_visualization_model.urdf (robot description, URDF)
Before this commit: robot end_effector_simple, 1 links, 0 joints
Links:
- link end_effector_simple: geometry visual sphere radius=0.0195

File: examples/push_T/urdf/sample_locations.urdf (robot description, URDF)
Before this commit: robot sample_sphere, 1 links, 0 joints
Links:
- link sample_sphere: geometry visual sphere radius=0.0195
