Commit message: misc changes

File: examples/trifinger/robot_properties_fingers/cube/HE_convex_terrain.urdf (robot description, URDF)
Before this commit: robot HE_sphere, 1 links, 0 joints
Links:
- link cube: mass 0.126919008388386 -> 0.233431934550168; geometry collision mesh filename=HE_convex_terrain.obj; visual mesh filename=HE_convex_terrain.obj
