Commit message: implemented python mesh sampling baseline

File: T_vertical_parametric.urdf (robot description, URDF)
Before this commit: robot cube, 4 links, 0 joints
Links:
- link body: geometry collision mesh filename=examples/sampling_c3/urdf/push_t_white.obj; visual mesh filename=examples/sampling_c3/urdf/push_t_white.obj
