Commit message: Update Trifinger example

File: examples/trifinger/robot_properties_fingers/urdf/trifinger.urdf (robot description, URDF)
Before this commit: robot finger_with_stage, 17 links, 16 joints
Links:
- removed link upper_holder_link
- added link trifinger_base_link, mass 1
- link finger_base_link_0: geometry collision mesh filename=meshes/base_back.obj scale=1 1 1; collision mesh filename=meshes/base_front.obj scale=1 1 1
- link finger_base_link_120: geometry collision mesh filename=meshes/base_back.obj scale=1 1 1; collision mesh filename=meshes/base_front.obj scale=1 1 1
- link finger_base_link_240: geometry collision mesh filename=meshes/base_back.obj scale=1 1 1; collision mesh filename=meshes/base_front.obj scale=1 1 1
- link finger_lower_link_0: mass 0.01 -> 0.035; geometry collision mesh filename=meshes/lower_link.obj scale=1 1 1; visual mesh filename=meshes/lower_link.obj scale=1 1 1
- link finger_lower_link_120: mass 0.01 -> 0.035; geometry collision mesh filename=meshes/lower_link.obj scale=1 1 1; visual mesh filename=meshes/lower_link.obj scale=1 1 1
- link finger_lower_link_240: mass 0.01 -> 0.035; geometry collision mesh filename=meshes/lower_link.obj scale=1 1 1; visual mesh filename=meshes/lower_link.obj scale=1 1 1
- link finger_middle_link_0: mass 0.2 -> 0.16; geometry collision mesh filename=meshes/middle_link.obj scale=1 1 1; visual mesh filename=meshes/middle_link.obj scale=1 1 1
- link finger_middle_link_120: mass 0.2 -> 0.16; geometry collision mesh filename=meshes/middle_link.obj scale=1 1 1; visual mesh filename=meshes/middle_link.obj scale=1 1 1
- link finger_middle_link_240: mass 0.2 -> 0.16; geometry collision mesh filename=meshes/middle_link.obj scale=1 1 1; visual mesh filename=meshes/middle_link.obj scale=1 1 1
- link finger_tip_link_0: mass 0.02 -> 0.01
- link finger_tip_link_120: mass 0.02 -> 0.01
- link finger_tip_link_240: mass 0.02 -> 0.01
- link finger_upper_link_0: mass 0.2 -> 0.157; geometry collision mesh filename=meshes/upper_link.obj scale=1 1 1; visual mesh filename=meshes/upper_link.obj scale=1 1 1
- link finger_upper_link_120: mass 0.2 -> 0.157; geometry collision mesh filename=meshes/upper_link.obj scale=1 1 1; visual mesh filename=meshes/upper_link.obj scale=1 1 1
- link finger_upper_link_240: mass 0.2 -> 0.157; geometry collision mesh filename=meshes/upper_link.obj scale=1 1 1; visual mesh filename=meshes/upper_link.obj scale=1 1 1
Joints:
- removed joint base_to_upper_holder_joint
- removed joint holder_to_finger_0
- removed joint holder_to_finger_120
- removed joint holder_to_finger_240
- added joint base_to_finger_0: type fixed, parent trifinger_base_link, child finger_base_link_0, origin xyz=-0.0395 0.0 0 rpy=0 0 0
- added joint base_to_finger_120: type fixed, parent trifinger_base_link, child finger_base_link_120, origin xyz=0.01975 0.034208 0 rpy=0 0 -2.0943951023931953
- added joint base_to_finger_240: type fixed, parent trifinger_base_link, child finger_base_link_240, origin xyz=0.01975 -0.034208 0 rpy=0 0 -4.1887902047863905
- added joint base_to_trifinger_base_joint: type fixed, parent base_link, child trifinger_base_link, origin xyz=0 0 0.282 rpy=0 0 -1.5707963267948966
- joint finger_base_to_upper_joint_0: axis 0 1 0 -> -1 0 0; limit lower=-1.5707963267948966 upper=1.5707963267948966 effort=1000 velocity=1000 -> lower=-1.5707963267948966 upper=1.5707963267948966 effort=0.36 velocity=20
- joint finger_base_to_upper_joint_120: axis 0 1 0 -> -1 0 0; limit lower=-1.5707963267948966 upper=1.5707963267948966 effort=1000 velocity=1000 -> lower=-1.5707963267948966 upper=1.5707963267948966 effort=0.36 velocity=20
- joint finger_base_to_upper_joint_240: axis 0 1 0 -> -1 0 0; limit lower=-1.5707963267948966 upper=1.5707963267948966 effort=1000 velocity=1000 -> lower=-1.5707963267948966 upper=1.5707963267948966 effort=0.36 velocity=20
- joint finger_lower_to_tip_joint_0: origin xyz=0 0 -0.16 -> xyz=0 -0.008 -0.16
- joint finger_lower_to_tip_joint_120: origin xyz=0 0 -0.16 -> xyz=0 -0.008 -0.16
- joint finger_lower_to_tip_joint_240: origin xyz=0 0 -0.16 -> xyz=0 -0.008 -0.16
- joint finger_middle_to_lower_joint_0: axis 1 0 0 -> 0 1 0; limit lower=-3.001966313430247 upper=3.001966313430247 effort=1000 velocity=1000 -> lower=-3.141592653589793 upper=3.141592653589793 effort=0.36 velocity=20; origin xyz=0 0 -0.16 rpy=0 0 0 -> xyz=0 -0.03745 -0.16 rpy=0 0 0
- joint finger_middle_to_lower_joint_120: axis 1 0 0 -> 0 1 0; limit lower=-3.001966313430247 upper=3.001966313430247 effort=1000 velocity=1000 -> lower=-3.141592653589793 upper=3.141592653589793 effort=0.36 velocity=20; origin xyz=0 0 -0.16 rpy=0 0 0 -> xyz=0 -0.03745 -0.16 rpy=0 0 0
- joint finger_middle_to_lower_joint_240: axis 1 0 0 -> 0 1 0; limit lower=-3.001966313430247 upper=3.001966313430247 effort=1000 velocity=1000 -> lower=-3.141592653589793 upper=3.141592653589793 effort=0.36 velocity=20; origin xyz=0 0 -0.16 rpy=0 0 0 -> xyz=0 -0.03745 -0.16 rpy=0 0 0
- joint finger_upper_to_middle_joint_0: axis -1 0 0 -> 0 1 0; limit lower=-1.3526301702956054 upper=4.494222823885399 effort=1000 velocity=1000 -> lower=-1.5707963267948966 upper=1.5707963267948966 effort=0.36 velocity=20; origin xyz=0 0 0 rpy=0 0 0 -> xyz=0 -0.014 0 rpy=0 0 0
- joint finger_upper_to_middle_joint_120: axis -1 0 0 -> 0 1 0; limit lower=-1.3526301702956054 upper=4.494222823885399 effort=1000 velocity=1000 -> lower=-1.5707963267948966 upper=1.5707963267948966 effort=0.36 velocity=20; origin xyz=0 0 0 rpy=0 0 0 -> xyz=0 -0.014 0 rpy=0 0 0
- joint finger_upper_to_middle_joint_240: axis -1 0 0 -> 0 1 0; limit lower=-1.3526301702956054 upper=4.494222823885399 effort=1000 velocity=1000 -> lower=-1.5707963267948966 upper=1.5707963267948966 effort=0.36 velocity=20; origin xyz=0 0 0 rpy=0 0 0 -> xyz=0 -0.014 0 rpy=0 0 0
