Commit message: chore: change frame name in scene urdf

File: examples/magna/urdf/common/scene.urdf (robot description, URDF)
Before this commit: robot round_belt_task_scene, 1 links, 0 joints
Links:
- removed link round_belt_task_scene
- added link scene; visual mesh filename=franka_mount/base_plate.obj; visual mesh filename=franka_mount/wooden_plate.gltf scale=0.001 0.001 0.001
