Commit message: feat: fix the script to generate urdf and implement the first simulation of the timing belt

File: examples/magna/urdf/timing_belt_task/timing_belt.urdf (robot description, URDF)
Before this commit: robot elliptical_belt, 269 links, 268 joints
Links:
- added link fb_rot_x
- added link fb_rot_y
- added link fb_trans_x
- added link fb_trans_y
- added link fb_trans_z
- added link timing_belt_base_link
- link dummy_0_1: mass 0.001 -> None
- link dummy_100_101: mass 0.001 -> None
- link dummy_101_102: mass 0.001 -> None
- link dummy_102_103: mass 0.001 -> None
- link dummy_103_104: mass 0.001 -> None
- link dummy_104_105: mass 0.001 -> None
- link dummy_105_106: mass 0.001 -> None
- link dummy_106_107: mass 0.001 -> None
- link dummy_107_108: mass 0.001 -> None
- link dummy_108_109: mass 0.001 -> None
- link dummy_109_110: mass 0.001 -> None
- link dummy_10_11: mass 0.001 -> None
- link dummy_110_111: mass 0.001 -> None
- link dummy_111_112: mass 0.001 -> None
- link dummy_112_113: mass 0.001 -> None
- link dummy_113_114: mass 0.001 -> None
- link dummy_114_115: mass 0.001 -> None
- link dummy_115_116: mass 0.001 -> None
- link dummy_116_117: mass 0.001 -> None
- link dummy_117_118: mass 0.001 -> None
- link dummy_118_119: mass 0.001 -> None
- link dummy_119_120: mass 0.001 -> None
- link dummy_11_12: mass 0.001 -> None
- link dummy_120_121: mass 0.001 -> None
- link dummy_121_122: mass 0.001 -> None
- link dummy_122_123: mass 0.001 -> None
- link dummy_123_124: mass 0.001 -> None
- link dummy_124_125: mass 0.001 -> None
- link dummy_125_126: mass 0.001 -> None
- link dummy_126_127: mass 0.001 -> None
- link dummy_127_128: mass 0.001 -> None
- link dummy_128_129: mass 0.001 -> None
- link dummy_129_130: mass 0.001 -> None
- link dummy_12_13: mass 0.001 -> None
- link dummy_130_131: mass 0.001 -> None
- link dummy_131_132: mass 0.001 -> None
- link dummy_132_133: mass 0.001 -> None
- link dummy_133_134: mass 0.001 -> None
- link dummy_13_14: mass 0.001 -> None
- link dummy_14_15: mass 0.001 -> None
- link dummy_15_16: mass 0.001 -> None
- link dummy_16_17: mass 0.001 -> None
- link dummy_17_18: mass 0.001 -> None
- link dummy_18_19: mass 0.001 -> None
- link dummy_19_20: mass 0.001 -> None
- link dummy_1_2: mass 0.001 -> None
- link dummy_20_21: mass 0.001 -> None
- link dummy_21_22: mass 0.001 -> None
- link dummy_22_23: mass 0.001 -> None
- link dummy_23_24: mass 0.001 -> None
- link dummy_24_25: mass 0.001 -> None
- link dummy_25_26: mass 0.001 -> None
- link dummy_26_27: mass 0.001 -> None
- link dummy_27_28: mass 0.001 -> None
- link dummy_28_29: mass 0.001 -> None
- link dummy_29_30: mass 0.001 -> None
- link dummy_2_3: mass 0.001 -> None
- link dummy_30_31: mass 0.001 -> None
- link dummy_31_32: mass 0.001 -> None
- link dummy_32_33: mass 0.001 -> None
- link dummy_33_34: mass 0.001 -> None
- link dummy_34_35: mass 0.001 -> None
- link dummy_35_36: mass 0.001 -> None
- link dummy_36_37: mass 0.001 -> None
- link dummy_37_38: mass 0.001 -> None
- link dummy_38_39: mass 0.001 -> None
- link dummy_39_40: mass 0.001 -> None
- link dummy_3_4: mass 0.001 -> None
- link dummy_40_41: mass 0.001 -> None
- link dummy_41_42: mass 0.001 -> None
- link dummy_42_43: mass 0.001 -> None
- link dummy_43_44: mass 0.001 -> None
- link dummy_44_45: mass 0.001 -> None
- link dummy_45_46: mass 0.001 -> None
- link dummy_46_47: mass 0.001 -> None
- link dummy_47_48: mass 0.001 -> None
- link dummy_48_49: mass 0.001 -> None
- link dummy_49_50: mass 0.001 -> None
- link dummy_4_5: mass 0.001 -> None
- link dummy_50_51: mass 0.001 -> None
- link dummy_51_52: mass 0.001 -> None
- link dummy_52_53: mass 0.001 -> None
- link dummy_53_54: mass 0.001 -> None
- link dummy_54_55: mass 0.001 -> None
- link dummy_55_56: mass 0.001 -> None
- link dummy_56_57: mass 0.001 -> None
- link dummy_57_58: mass 0.001 -> None
- link dummy_58_59: mass 0.001 -> None
- link dummy_59_60: mass 0.001 -> None
- link dummy_5_6: mass 0.001 -> None
- link dummy_60_61: mass 0.001 -> None
- link dummy_61_62: mass 0.001 -> None
- link dummy_62_63: mass 0.001 -> None
- link dummy_63_64: mass 0.001 -> None
- link dummy_64_65: mass 0.001 -> None
- link dummy_65_66: mass 0.001 -> None
- link dummy_66_67: mass 0.001 -> None
- link dummy_67_68: mass 0.001 -> None
- link dummy_68_69: mass 0.001 -> None
- link dummy_69_70: mass 0.001 -> None
- link dummy_6_7: mass 0.001 -> None
- link dummy_70_71: mass 0.001 -> None
- link dummy_71_72: mass 0.001 -> None
- link dummy_72_73: mass 0.001 -> None
- link dummy_73_74: mass 0.001 -> None
- link dummy_74_75: mass 0.001 -> None
- link dummy_75_76: mass 0.001 -> None
- link dummy_76_77: mass 0.001 -> None
- link dummy_77_78: mass 0.001 -> None
- link dummy_78_79: mass 0.001 -> None
- link dummy_79_80: mass 0.001 -> None
- link dummy_7_8: mass 0.001 -> None
- link dummy_80_81: mass 0.001 -> None
- link dummy_81_82: mass 0.001 -> None
- link dummy_82_83: mass 0.001 -> None
- link dummy_83_84: mass 0.001 -> None
- link dummy_84_85: mass 0.001 -> None
- link dummy_85_86: mass 0.001 -> None
- link dummy_86_87: mass 0.001 -> None
- link dummy_87_88: mass 0.001 -> None
- link dummy_88_89: mass 0.001 -> None
- link dummy_89_90: mass 0.001 -> None
- link dummy_8_9: mass 0.001 -> None
- link dummy_90_91: mass 0.001 -> None
- link dummy_91_92: mass 0.001 -> None
- link dummy_92_93: mass 0.001 -> None
- link dummy_93_94: mass 0.001 -> None
- link dummy_94_95: mass 0.001 -> None
- link dummy_95_96: mass 0.001 -> None
- link dummy_96_97: mass 0.001 -> None
- link dummy_97_98: mass 0.001 -> None
- link dummy_98_99: mass 0.001 -> None
- link dummy_99_100: mass 0.001 -> None
- link dummy_9_10: mass 0.001 -> None
Joints:
- added joint float_joint_pitch: type revolute, parent fb_rot_x, child fb_rot_y, origin xyz=0.000000 0.000000 0.000000 rpy=0.000000 0.000000 0.000000, axis 0 1 0, limit lower=-1.57 upper=1.57 effort=1000 velocity=100
- added joint float_joint_roll: type revolute, parent fb_trans_z, child fb_rot_x, origin xyz=0.000000 0.000000 0.000000 rpy=0.000000 0.000000 0.000000, axis 1 0 0, limit lower=-1.57 upper=1.57 effort=1000 velocity=100
- added joint float_joint_x: type prismatic, parent timing_belt_base_link, child fb_trans_x, origin xyz=0.000000 0.000000 0.000000 rpy=0.000000 0.000000 0.000000, axis 1 0 0, limit lower=-1.57 upper=1.57 effort=1000 velocity=100
- added joint float_joint_y: type prismatic, parent fb_trans_x, child fb_trans_y, origin xyz=0.000000 0.000000 0.000000 rpy=0.000000 0.000000 0.000000, axis 0 1 0, limit lower=-1.57 upper=1.57 effort=1000 velocity=100
- added joint float_joint_yaw: type revolute, parent fb_rot_y, child rod_0, origin xyz=0.000000 0.000000 0.000000 rpy=0.000000 0.000000 0.000000, axis 0 0 1, limit lower=-1.57 upper=1.57 effort=1000 velocity=100
- added joint float_joint_z: type prismatic, parent fb_trans_y, child fb_trans_z, origin xyz=0.000000 0.000000 0.000000 rpy=0.000000 0.000000 0.000000, axis 0 0 1, limit lower=-1.57 upper=1.57 effort=1000 velocity=100

Commit message: feat: add torsional springs to revolute joints in the timing belt model

File: examples/magna/urdf/timing_belt_task/timing_belt.urdf (robot description, URDF)
Before this commit: robot timing_belt, 275 links, 274 joints
Links:
- removed link fb_rot_x
- removed link fb_rot_y
- removed link fb_trans_x
- removed link fb_trans_y
- removed link fb_trans_z
- removed link timing_belt_base_link
Joints:
- removed joint float_joint_pitch
- removed joint float_joint_roll
- removed joint float_joint_x
- removed joint float_joint_y
- removed joint float_joint_yaw
- removed joint float_joint_z
