Commit message: fix: reduce the number of timing belt element to speed up the simulation

File: examples/magna/urdf/timing_belt_task/timing_belt.urdf (robot description, URDF)
Before this commit: robot timing_belt, 269 links, 268 joints
Links:
- removed link dummy_100_101
- removed link dummy_101_102
- removed link dummy_102_103
- removed link dummy_103_104
- removed link dummy_104_105
- removed link dummy_105_106
- removed link dummy_106_107
- removed link dummy_107_108
- removed link dummy_108_109
- removed link dummy_109_110
- removed link dummy_110_111
- removed link dummy_111_112
- removed link dummy_112_113
- removed link dummy_113_114
- removed link dummy_114_115
- removed link dummy_115_116
- removed link dummy_116_117
- removed link dummy_117_118
- removed link dummy_118_119
- removed link dummy_119_120
- removed link dummy_120_121
- removed link dummy_121_122
- removed link dummy_122_123
- removed link dummy_123_124
- removed link dummy_124_125
- removed link dummy_125_126
- removed link dummy_126_127
- removed link dummy_127_128
- removed link dummy_128_129
- removed link dummy_129_130
- removed link dummy_130_131
- removed link dummy_131_132
- removed link dummy_132_133
- removed link dummy_133_134
- removed link dummy_67_68
- removed link dummy_68_69
- removed link dummy_69_70
- removed link dummy_70_71
- removed link dummy_71_72
- removed link dummy_72_73
- removed link dummy_73_74
- removed link dummy_74_75
- removed link dummy_75_76
- removed link dummy_76_77
- removed link dummy_77_78
- removed link dummy_78_79
- removed link dummy_79_80
- removed link dummy_80_81
- removed link dummy_81_82
- removed link dummy_82_83
- removed link dummy_83_84
- removed link dummy_84_85
- removed link dummy_85_86
- removed link dummy_86_87
- removed link dummy_87_88
- removed link dummy_88_89
- removed link dummy_89_90
- removed link dummy_90_91
- removed link dummy_91_92
- removed link dummy_92_93
- removed link dummy_93_94
- removed link dummy_94_95
- removed link dummy_95_96
- removed link dummy_96_97
- removed link dummy_97_98
- removed link dummy_98_99
- removed link dummy_99_100
- removed link rod_100
- removed link rod_101
- removed link rod_102
- removed link rod_103
- removed link rod_104
- removed link rod_105
- removed link rod_106
- removed link rod_107
- removed link rod_108
- removed link rod_109
- removed link rod_110
- removed link rod_111
- removed link rod_112
- removed link rod_113
- removed link rod_114
- removed link rod_115
- removed link rod_116
- removed link rod_117
- removed link rod_118
- removed link rod_119
- removed link rod_120
- removed link rod_121
- removed link rod_122
- removed link rod_123
- removed link rod_124
- removed link rod_125
- removed link rod_126
- removed link rod_127
- removed link rod_128
- removed link rod_129
- removed link rod_130
- removed link rod_131
- removed link rod_132
- removed link rod_133
- removed link rod_134
- removed link rod_68
- removed link rod_69
- removed link rod_70
- removed link rod_71
- removed link rod_72
- removed link rod_73
- removed link rod_74
- removed link rod_75
- removed link rod_76
- removed link rod_77
- removed link rod_78
- removed link rod_79
- removed link rod_80
- removed link rod_81
- removed link rod_82
- removed link rod_83
- removed link rod_84
- removed link rod_85
- removed link rod_86
- removed link rod_87
- removed link rod_88
- removed link rod_89
- removed link rod_90
- removed link rod_91
- removed link rod_92
- removed link rod_93
- removed link rod_94
- removed link rod_95
- removed link rod_96
- removed link rod_97
- removed link rod_98
- removed link rod_99
- link rod_0: geometry collision box size=0.0045 0.0022 0.025; visual box size=0.0045 0.0022 0.025
- link rod_1: geometry collision box size=0.009 0.0022 0.025; visual box size=0.009 0.0022 0.025
- link rod_10: geometry collision box size=0.009 0.0022 0.025; visual box size=0.009 0.0022 0.025
- link rod_11: geometry collision box size=0.009 0.0022 0.025; visual box size=0.009 0.0022 0.025
- link rod_12: geometry collision box size=0.009 0.0022 0.025; visual box size=0.009 0.0022 0.025
- link rod_13: geometry collision box size=0.009 0.0022 0.025; visual box size=0.009 0.0022 0.025
- link rod_14: geometry collision box size=0.009 0.0022 0.025; visual box size=0.009 0.0022 0.025
- link rod_15: geometry collision box size=0.009 0.0022 0.025; visual box size=0.009 0.0022 0.025
- link rod_16: geometry collision box size=0.009 0.0022 0.025; visual box size=0.009 0.0022 0.025
- link rod_17: geometry collision box size=0.009 0.0022 0.025; visual box size=0.009 0.0022 0.025
- link rod_18: geometry collision box size=0.009 0.0022 0.025; visual box size=0.009 0.0022 0.025
- link rod_19: geometry collision box size=0.009 0.0022 0.025; visual box size=0.009 0.0022 0.025
- link rod_2: geometry collision box size=0.009 0.0022 0.025; visual box size=0.009 0.0022 0.025
- link rod_20: geometry collision box size=0.009 0.0022 0.025; visual box size=0.009 0.0022 0.025
- link rod_21: geometry collision box size=0.009 0.0022 0.025; visual box size=0.009 0.0022 0.025
- link rod_22: geometry collision box size=0.009 0.0022 0.025; visual box size=0.009 0.0022 0.025
- link rod_23: geometry collision box size=0.009 0.0022 0.025; visual box size=0.009 0.0022 0.025
- link rod_24: geometry collision box size=0.009 0.0022 0.025; visual box size=0.009 0.0022 0.025
- link rod_25: geometry collision box size=0.009 0.0022 0.025; visual box size=0.009 0.0022 0.025
- link rod_26: geometry collision box size=0.009 0.0022 0.025; visual box size=0.009 0.0022 0.025
- link rod_27: geometry collision box size=0.009 0.0022 0.025; visual box size=0.009 0.0022 0.025
- link rod_28: geometry collision box size=0.009 0.0022 0.025; visual box size=0.009 0.0022 0.025
- link rod_29: geometry collision box size=0.009 0.0022 0.025; visual box size=0.009 0.0022 0.025
- link rod_3: geometry collision box size=0.009 0.0022 0.025; visual box size=0.009 0.0022 0.025
- link rod_30: geometry collision box size=0.009 0.0022 0.025; visual box size=0.009 0.0022 0.025
- link rod_31: geometry collision box size=0.009 0.0022 0.025; visual box size=0.009 0.0022 0.025
- link rod_32: geometry collision box size=0.009 0.0022 0.025; visual box size=0.009 0.0022 0.025
- link rod_33: geometry collision box size=0.009 0.0022 0.025; visual box size=0.009 0.0022 0.025
- link rod_34: geometry collision box size=0.009 0.0022 0.025; visual box size=0.009 0.0022 0.025
- link rod_35: geometry collision box size=0.009 0.0022 0.025; visual box size=0.009 0.0022 0.025
- link rod_36: geometry collision box size=0.009 0.0022 0.025; visual box size=0.009 0.0022 0.025
- link rod_37: geometry collision box size=0.009 0.0022 0.025; visual box size=0.009 0.0022 0.025
- link rod_38: geometry collision box size=0.009 0.0022 0.025; visual box size=0.009 0.0022 0.025
- link rod_39: geometry collision box size=0.009 0.0022 0.025; visual box size=0.009 0.0022 0.025
- link rod_4: geometry collision box size=0.009 0.0022 0.025; visual box size=0.009 0.0022 0.025
- link rod_40: geometry collision box size=0.009 0.0022 0.025; visual box size=0.009 0.0022 0.025
- link rod_41: geometry collision box size=0.009 0.0022 0.025; visual box size=0.009 0.0022 0.025
- link rod_42: geometry collision box size=0.009 0.0022 0.025; visual box size=0.009 0.0022 0.025
- link rod_43: geometry collision box size=0.009 0.0022 0.025; visual box size=0.009 0.0022 0.025
- link rod_44: geometry collision box size=0.009 0.0022 0.025; visual box size=0.009 0.0022 0.025
- link rod_45: geometry collision box size=0.009 0.0022 0.025; visual box size=0.009 0.0022 0.025
- link rod_46: geometry collision box size=0.009 0.0022 0.025; visual box size=0.009 0.0022 0.025
- link rod_47: geometry collision box size=0.009 0.0022 0.025; visual box size=0.009 0.0022 0.025
- link rod_48: geometry collision box size=0.009 0.0022 0.025; visual box size=0.009 0.0022 0.025
- link rod_49: geometry collision box size=0.009 0.0022 0.025; visual box size=0.009 0.0022 0.025
- link rod_5: geometry collision box size=0.009 0.0022 0.025; visual box size=0.009 0.0022 0.025
- link rod_50: geometry collision box size=0.009 0.0022 0.025; visual box size=0.009 0.0022 0.025
- link rod_51: geometry collision box size=0.009 0.0022 0.025; visual box size=0.009 0.0022 0.025
- link rod_52: geometry collision box size=0.009 0.0022 0.025; visual box size=0.009 0.0022 0.025
- link rod_53: geometry collision box size=0.009 0.0022 0.025; visual box size=0.009 0.0022 0.025
- link rod_54: geometry collision box size=0.009 0.0022 0.025; visual box size=0.009 0.0022 0.025
- link rod_55: geometry collision box size=0.009 0.0022 0.025; visual box size=0.009 0.0022 0.025
- link rod_56: geometry collision box size=0.009 0.0022 0.025; visual box size=0.009 0.0022 0.025
- link rod_57: geometry collision box size=0.009 0.0022 0.025; visual box size=0.009 0.0022 0.025
- link rod_58: geometry collision box size=0.009 0.0022 0.025; visual box size=0.009 0.0022 0.025
- link rod_59: geometry collision box size=0.009 0.0022 0.025; visual box size=0.009 0.0022 0.025
- link rod_6: geometry collision box size=0.009 0.0022 0.025; visual box size=0.009 0.0022 0.025
- link rod_60: geometry collision box size=0.009 0.0022 0.025; visual box size=0.009 0.0022 0.025
- link rod_61: geometry collision box size=0.009 0.0022 0.025; visual box size=0.009 0.0022 0.025
- link rod_62: geometry collision box size=0.009 0.0022 0.025; visual box size=0.009 0.0022 0.025
- link rod_63: geometry collision box size=0.009 0.0022 0.025; visual box size=0.009 0.0022 0.025
- link rod_64: geometry collision box size=0.009 0.0022 0.025; visual box size=0.009 0.0022 0.025
- link rod_65: geometry collision box size=0.009 0.0022 0.025; visual box size=0.009 0.0022 0.025
- link rod_66: geometry collision box size=0.009 0.0022 0.025; visual box size=0.009 0.0022 0.025
- link rod_67: mass 0.001 -> 0.0005; geometry collision box size=0.0045 0.0022 0.025; visual box size=0.0045 0.0022 0.025
- link rod_7: geometry collision box size=0.009 0.0022 0.025; visual box size=0.009 0.0022 0.025
- link rod_8: geometry collision box size=0.009 0.0022 0.025; visual box size=0.009 0.0022 0.025
- link rod_9: geometry collision box size=0.009 0.0022 0.025; visual box size=0.009 0.0022 0.025
Joints:
- removed joint joint_100_roll
- removed joint joint_100_yaw
- removed joint joint_101_roll
- removed joint joint_101_yaw
- removed joint joint_102_roll
- removed joint joint_102_yaw
- removed joint joint_103_roll
- removed joint joint_103_yaw
- removed joint joint_104_roll
- removed joint joint_104_yaw
- removed joint joint_105_roll
- removed joint joint_105_yaw
- removed joint joint_106_roll
- removed joint joint_106_yaw
- removed joint joint_107_roll
- removed joint joint_107_yaw
- removed joint joint_108_roll
- removed joint joint_108_yaw
- removed joint joint_109_roll
- removed joint joint_109_yaw
- removed joint joint_110_roll
- removed joint joint_110_yaw
- removed joint joint_111_roll
- removed joint joint_111_yaw
- removed joint joint_112_roll
- removed joint joint_112_yaw
- removed joint joint_113_roll
- removed joint joint_113_yaw
- removed joint joint_114_roll
- removed joint joint_114_yaw
- removed joint joint_115_roll
- removed joint joint_115_yaw
- removed joint joint_116_roll
- removed joint joint_116_yaw
- removed joint joint_117_roll
- removed joint joint_117_yaw
- removed joint joint_118_roll
- removed joint joint_118_yaw
- removed joint joint_119_roll
- removed joint joint_119_yaw
- removed joint joint_120_roll
- removed joint joint_120_yaw
- removed joint joint_121_roll
- removed joint joint_121_yaw
- removed joint joint_122_roll
- removed joint joint_122_yaw
- removed joint joint_123_roll
- removed joint joint_123_yaw
- removed joint joint_124_roll
- removed joint joint_124_yaw
- removed joint joint_125_roll
- removed joint joint_125_yaw
- removed joint joint_126_roll
- removed joint joint_126_yaw
- removed joint joint_127_roll
- removed joint joint_127_yaw
- removed joint joint_128_roll
- removed joint joint_128_yaw
- removed joint joint_129_roll
- removed joint joint_129_yaw
- removed joint joint_130_roll
- removed joint joint_130_yaw
- removed joint joint_131_roll
- removed joint joint_131_yaw
- removed joint joint_132_roll
- removed joint joint_132_yaw
- removed joint joint_133_roll
- removed joint joint_133_yaw
- removed joint joint_67_roll
- removed joint joint_67_yaw
- removed joint joint_68_roll
- removed joint joint_68_yaw
- removed joint joint_69_roll
- removed joint joint_69_yaw
- removed joint joint_70_roll
- removed joint joint_70_yaw
- removed joint joint_71_roll
- removed joint joint_71_yaw
- removed joint joint_72_roll
- removed joint joint_72_yaw
- removed joint joint_73_roll
- removed joint joint_73_yaw
- removed joint joint_74_roll
- removed joint joint_74_yaw
- removed joint joint_75_roll
- removed joint joint_75_yaw
- removed joint joint_76_roll
- removed joint joint_76_yaw
- removed joint joint_77_roll
- removed joint joint_77_yaw
- removed joint joint_78_roll
- removed joint joint_78_yaw
- removed joint joint_79_roll
- removed joint joint_79_yaw
- removed joint joint_80_roll
- removed joint joint_80_yaw
- removed joint joint_81_roll
- removed joint joint_81_yaw
- removed joint joint_82_roll
- removed joint joint_82_yaw
- removed joint joint_83_roll
- removed joint joint_83_yaw
- removed joint joint_84_roll
- removed joint joint_84_yaw
- removed joint joint_85_roll
- removed joint joint_85_yaw
- removed joint joint_86_roll
- removed joint joint_86_yaw
- removed joint joint_87_roll
- removed joint joint_87_yaw
- removed joint joint_88_roll
- removed joint joint_88_yaw
- removed joint joint_89_roll
- removed joint joint_89_yaw
- removed joint joint_90_roll
- removed joint joint_90_yaw
- removed joint joint_91_roll
- removed joint joint_91_yaw
- removed joint joint_92_roll
- removed joint joint_92_yaw
- removed joint joint_93_roll
- removed joint joint_93_yaw
- removed joint joint_94_roll
- removed joint joint_94_yaw
- removed joint joint_95_roll
- removed joint joint_95_yaw
- removed joint joint_96_roll
- removed joint joint_96_yaw
- removed joint joint_97_roll
- removed joint joint_97_yaw
- removed joint joint_98_roll
- removed joint joint_98_yaw
- removed joint joint_99_roll
- removed joint joint_99_yaw
- joint joint_0_yaw: origin xyz=0.004591 0.000225 0.000000 rpy=0.000000 0.000000 0.097815 -> xyz=0.009920 0.001003 0.000000 rpy=0.000000 0.000000 0.200333
- joint joint_10_yaw: origin xyz=0.004596 0.000125 0.000000 rpy=0.000000 0.000000 0.053882 -> xyz=0.009981 0.000299 0.000000 rpy=0.000000 0.000000 0.059193
- joint joint_11_yaw: origin xyz=0.004597 0.000117 0.000000 rpy=0.000000 0.000000 0.050146 -> xyz=0.009982 0.000279 0.000000 rpy=0.000000 0.000000 0.055304
- joint joint_12_yaw: origin xyz=0.004597 0.000109 0.000000 rpy=0.000000 0.000000 0.046807 -> xyz=0.009982 0.000263 0.000000 rpy=0.000000 0.000000 0.052347
- joint joint_13_yaw: origin xyz=0.004597 0.000102 0.000000 rpy=0.000000 0.000000 0.043835 -> xyz=0.009983 0.000252 0.000000 rpy=0.000000 0.000000 0.050164
- joint joint_14_yaw: origin xyz=0.004597 0.000096 0.000000 rpy=0.000000 0.000000 0.041197 -> xyz=0.009983 0.000244 0.000000 rpy=0.000000 0.000000 0.048642
- joint joint_15_yaw: origin xyz=0.004597 0.000090 0.000000 rpy=0.000000 0.000000 0.038860 -> xyz=0.009983 0.000239 0.000000 rpy=0.000000 0.000000 0.047706
- joint joint_16_yaw: origin xyz=0.004597 0.000085 0.000000 rpy=0.000000 0.000000 0.036790 -> xyz=0.009983 0.000236 0.000000 rpy=0.000000 0.000000 0.047313
- joint joint_17_yaw: origin xyz=0.004598 0.000081 0.000000 rpy=0.000000 0.000000 0.034959 -> xyz=0.009983 0.000237 0.000000 rpy=0.000000 0.000000 0.047444
- joint joint_18_yaw: origin xyz=0.004598 0.000077 0.000000 rpy=0.000000 0.000000 0.033339 -> xyz=0.009983 0.000239 0.000000 rpy=0.000000 0.000000 0.048104
- joint joint_19_yaw: origin xyz=0.004598 0.000074 0.000000 rpy=0.000000 0.000000 0.031907 -> xyz=0.009983 0.000245 0.000000 rpy=0.000000 0.000000 0.049325
- joint joint_1_yaw: origin xyz=0.004591 0.000222 0.000000 rpy=0.000000 0.000000 0.096142 -> xyz=0.009927 0.000945 0.000000 rpy=0.000000 0.000000 0.186647
- joint joint_20_yaw: origin xyz=0.004598 0.000071 0.000000 rpy=0.000000 0.000000 0.030642 -> xyz=0.009983 0.000254 0.000000 rpy=0.000000 0.000000 0.051167
- joint joint_21_yaw: origin xyz=0.004598 0.000068 0.000000 rpy=0.000000 0.000000 0.029527 -> xyz=0.009982 0.000266 0.000000 rpy=0.000000 0.000000 0.053720
- joint joint_22_yaw: origin xyz=0.004598 0.000066 0.000000 rpy=0.000000 0.000000 0.028547 -> xyz=0.009981 0.000282 0.000000 rpy=0.000000 0.000000 0.057120
- joint joint_23_yaw: origin xyz=0.004598 0.000064 0.000000 rpy=0.000000 0.000000 0.027687 -> xyz=0.009981 0.000303 0.000000 rpy=0.000000 0.000000 0.061553
- joint joint_24_yaw: origin xyz=0.004598 0.000062 0.000000 rpy=0.000000 0.000000 0.026937 -> xyz=0.009979 0.000330 0.000000 rpy=0.000000 0.000000 0.067281
- joint joint_25_yaw: origin xyz=0.004598 0.000061 0.000000 rpy=0.000000 0.000000 0.026287 -> xyz=0.009978 0.000366 0.000000 rpy=0.000000 0.000000 0.074652
- joint joint_26_yaw: origin xyz=0.004598 0.000059 0.000000 rpy=0.000000 0.000000 0.025729 -> xyz=0.009975 0.000411 0.000000 rpy=0.000000 0.000000 0.084130
- joint joint_27_yaw: origin xyz=0.004598 0.000058 0.000000 rpy=0.000000 0.000000 0.025256 -> xyz=0.009972 0.000469 0.000000 rpy=0.000000 0.000000 0.096285
- joint joint_28_yaw: origin xyz=0.004598 0.000057 0.000000 rpy=0.000000 0.000000 0.024863 -> xyz=0.009967 0.000543 0.000000 rpy=0.000000 0.000000 0.111728
- joint joint_29_yaw: origin xyz=0.004598 0.000057 0.000000 rpy=0.000000 0.000000 0.024544 -> xyz=0.009959 0.000635 0.000000 rpy=0.000000 0.000000 0.130858
- joint joint_2_yaw: origin xyz=0.004592 0.000215 0.000000 rpy=0.000000 0.000000 0.092993 -> xyz=0.009940 0.000841 0.000000 rpy=0.000000 0.000000 0.164954
- joint joint_30_yaw: origin xyz=0.004598 0.000056 0.000000 rpy=0.000000 0.000000 0.024296 -> xyz=0.009949 0.000744 0.000000 rpy=0.000000 0.000000 0.153217
- joint joint_31_yaw: origin xyz=0.004598 0.000056 0.000000 rpy=0.000000 0.000000 0.024117 -> xyz=0.009937 0.000860 0.000000 rpy=0.000000 0.000000 0.176356
- joint joint_32_yaw: origin xyz=0.004598 0.000055 0.000000 rpy=0.000000 0.000000 0.024003 -> xyz=0.009925 0.000959 0.000000 rpy=0.000000 0.000000 0.194930
- joint joint_33_yaw: origin xyz=0.004598 0.000055 0.000000 rpy=0.000000 0.000000 0.023955 -> xyz=0.009919 0.001006 0.000000 rpy=0.000000 0.000000 0.202214
- joint joint_34_yaw: origin xyz=0.004598 0.000055 0.000000 rpy=0.000000 0.000000 0.023971 -> xyz=0.009923 0.000982 0.000000 rpy=0.000000 0.000000 0.194930
- joint joint_35_yaw: origin xyz=0.004598 0.000055 0.000000 rpy=0.000000 0.000000 0.024052 -> xyz=0.009934 0.000897 0.000000 rpy=0.000000 0.000000 0.176356
- joint joint_36_yaw: origin xyz=0.004598 0.000056 0.000000 rpy=0.000000 0.000000 0.024198 -> xyz=0.009946 0.000783 0.000000 rpy=0.000000 0.000000 0.153217
- joint joint_37_yaw: origin xyz=0.004598 0.000056 0.000000 rpy=0.000000 0.000000 0.024411 -> xyz=0.009957 0.000670 0.000000 rpy=0.000000 0.000000 0.130858
- joint joint_38_yaw: origin xyz=0.004598 0.000057 0.000000 rpy=0.000000 0.000000 0.024694 -> xyz=0.009965 0.000572 0.000000 rpy=0.000000 0.000000 0.111728
- joint joint_39_yaw: origin xyz=0.004598 0.000057 0.000000 rpy=0.000000 0.000000 0.025050 -> xyz=0.009971 0.000492 0.000000 rpy=0.000000 0.000000 0.096285
- joint joint_3_yaw: origin xyz=0.004592 0.000206 0.000000 rpy=0.000000 0.000000 0.088706 -> xyz=0.009952 0.000725 0.000000 rpy=0.000000 0.000000 0.141725
- joint joint_40_yaw: origin xyz=0.004598 0.000058 0.000000 rpy=0.000000 0.000000 0.025482 -> xyz=0.009975 0.000429 0.000000 rpy=0.000000 0.000000 0.084130
- joint joint_41_yaw: origin xyz=0.004598 0.000060 0.000000 rpy=0.000000 0.000000 0.025997 -> xyz=0.009977 0.000380 0.000000 rpy=0.000000 0.000000 0.074652
- joint joint_42_yaw: origin xyz=0.004598 0.000061 0.000000 rpy=0.000000 0.000000 0.026600 -> xyz=0.009979 0.000341 0.000000 rpy=0.000000 0.000000 0.067281
- joint joint_43_yaw: origin xyz=0.004598 0.000062 0.000000 rpy=0.000000 0.000000 0.027299 -> xyz=0.009980 0.000311 0.000000 rpy=0.000000 0.000000 0.061553
- joint joint_44_yaw: origin xyz=0.004598 0.000064 0.000000 rpy=0.000000 0.000000 0.028103 -> xyz=0.009981 0.000288 0.000000 rpy=0.000000 0.000000 0.057120
- joint joint_45_yaw: origin xyz=0.004598 0.000066 0.000000 rpy=0.000000 0.000000 0.029021 -> xyz=0.009982 0.000271 0.000000 rpy=0.000000 0.000000 0.053720
- joint joint_46_yaw: origin xyz=0.004598 0.000069 0.000000 rpy=0.000000 0.000000 0.030067 -> xyz=0.009982 0.000257 0.000000 rpy=0.000000 0.000000 0.051167
- joint joint_47_yaw: origin xyz=0.004598 0.000071 0.000000 rpy=0.000000 0.000000 0.031255 -> xyz=0.009983 0.000248 0.000000 rpy=0.000000 0.000000 0.049325
- joint joint_48_yaw: origin xyz=0.004598 0.000074 0.000000 rpy=0.000000 0.000000 0.032600 -> xyz=0.009983 0.000241 0.000000 rpy=0.000000 0.000000 0.048104
- joint joint_49_yaw: origin xyz=0.004598 0.000078 0.000000 rpy=0.000000 0.000000 0.034124 -> xyz=0.009983 0.000237 0.000000 rpy=0.000000 0.000000 0.047444
- joint joint_4_yaw: origin xyz=0.004593 0.000194 0.000000 rpy=0.000000 0.000000 0.083678 -> xyz=0.009962 0.000619 0.000000 rpy=0.000000 0.000000 0.120830
- joint joint_50_yaw: origin xyz=0.004598 0.000082 0.000000 rpy=0.000000 0.000000 0.035846 -> xyz=0.009983 0.000236 0.000000 rpy=0.000000 0.000000 0.047313
- joint joint_51_yaw: origin xyz=0.004597 0.000086 0.000000 rpy=0.000000 0.000000 0.037793 -> xyz=0.009983 0.000238 0.000000 rpy=0.000000 0.000000 0.047706
- joint joint_52_yaw: origin xyz=0.004597 0.000091 0.000000 rpy=0.000000 0.000000 0.039993 -> xyz=0.009983 0.000242 0.000000 rpy=0.000000 0.000000 0.048642
- joint joint_53_yaw: origin xyz=0.004597 0.000097 0.000000 rpy=0.000000 0.000000 0.042477 -> xyz=0.009983 0.000249 0.000000 rpy=0.000000 0.000000 0.050164
- joint joint_54_yaw: origin xyz=0.004597 0.000103 0.000000 rpy=0.000000 0.000000 0.045277 -> xyz=0.009982 0.000259 0.000000 rpy=0.000000 0.000000 0.052347
- joint joint_55_yaw: origin xyz=0.004597 0.000110 0.000000 rpy=0.000000 0.000000 0.048428 -> xyz=0.009982 0.000273 0.000000 rpy=0.000000 0.000000 0.055304
- joint joint_56_yaw: origin xyz=0.004596 0.000118 0.000000 rpy=0.000000 0.000000 0.051963 -> xyz=0.009981 0.000292 0.000000 rpy=0.000000 0.000000 0.059193
- joint joint_57_yaw: origin xyz=0.004596 0.000127 0.000000 rpy=0.000000 0.000000 0.055906 -> xyz=0.009980 0.000316 0.000000 rpy=0.000000 0.000000 0.064236
- joint joint_58_yaw: origin xyz=0.004596 0.000137 0.000000 rpy=0.000000 0.000000 0.060270 -> xyz=0.009979 0.000347 0.000000 rpy=0.000000 0.000000 0.070735
- joint joint_59_yaw: origin xyz=0.004595 0.000148 0.000000 rpy=0.000000 0.000000 0.065043 -> xyz=0.009977 0.000387 0.000000 rpy=0.000000 0.000000 0.079095
- joint joint_5_yaw: origin xyz=0.004594 0.000182 0.000000 rpy=0.000000 0.000000 0.078287 -> xyz=0.009968 0.000529 0.000000 rpy=0.000000 0.000000 0.103561
- joint joint_60_yaw: origin xyz=0.004595 0.000159 0.000000 rpy=0.000000 0.000000 0.070173 -> xyz=0.009974 0.000438 0.000000 rpy=0.000000 0.000000 0.089834
- joint joint_61_yaw: origin xyz=0.004594 0.000172 0.000000 rpy=0.000000 0.000000 0.075555 -> xyz=0.009970 0.000504 0.000000 rpy=0.000000 0.000000 0.103561
- joint joint_62_yaw: origin xyz=0.004594 0.000184 0.000000 rpy=0.000000 0.000000 0.081006 -> xyz=0.009964 0.000587 0.000000 rpy=0.000000 0.000000 0.120830
- joint joint_63_yaw: origin xyz=0.004593 0.000196 0.000000 rpy=0.000000 0.000000 0.086259 -> xyz=0.009955 0.000688 0.000000 rpy=0.000000 0.000000 0.141725
- joint joint_64_yaw: origin xyz=0.004592 0.000207 0.000000 rpy=0.000000 0.000000 0.090967 -> xyz=0.009943 0.000802 0.000000 rpy=0.000000 0.000000 0.164954
- joint joint_65_yaw: origin xyz=0.004592 0.000216 0.000000 rpy=0.000000 0.000000 0.094733 -> xyz=0.009930 0.000914 0.000000 rpy=0.000000 0.000000 0.186647
- joint joint_66_yaw: origin xyz=0.004591 0.000223 0.000000 rpy=0.000000 0.000000 0.097179 -> xyz=0.009921 0.000991 0.000000 rpy=0.000000 0.000000 0.200333
- joint joint_6_yaw: origin xyz=0.004594 0.000169 0.000000 rpy=0.000000 0.000000 0.072842 -> xyz=0.009973 0.000458 0.000000 rpy=0.000000 0.000000 0.089834
- joint joint_7_yaw: origin xyz=0.004595 0.000157 0.000000 rpy=0.000000 0.000000 0.067568 -> xyz=0.009976 0.000403 0.000000 rpy=0.000000 0.000000 0.079095
- joint joint_8_yaw: origin xyz=0.004595 0.000146 0.000000 rpy=0.000000 0.000000 0.062607 -> xyz=0.009978 0.000359 0.000000 rpy=0.000000 0.000000 0.070735
- joint joint_9_yaw: origin xyz=0.004596 0.000135 0.000000 rpy=0.000000 0.000000 0.058035 -> xyz=0.009980 0.000325 0.000000 rpy=0.000000 0.000000 0.064236
