Commit message: fix: adjust the circumference of the timing belt based on real measurements

File: examples/magna/urdf/timing_belt_task/timing_belt.urdf (robot description, URDF)
Before this commit: robot timing_belt, 135 links, 134 joints
Joints:
- joint joint_0_yaw: origin xyz=0.009920 0.001003 0.000000 rpy=0.000000 0.000000 0.200333 -> xyz=0.010219 0.001114 0.000000 rpy=0.000000 0.000000 0.215536
- joint joint_10_yaw: origin xyz=0.009981 0.000299 0.000000 rpy=0.000000 0.000000 0.059193 -> xyz=0.010294 0.000293 0.000000 rpy=0.000000 0.000000 0.056137
- joint joint_11_yaw: origin xyz=0.009982 0.000279 0.000000 rpy=0.000000 0.000000 0.055304 -> xyz=0.010294 0.000272 0.000000 rpy=0.000000 0.000000 0.052331
- joint joint_12_yaw: origin xyz=0.009982 0.000263 0.000000 rpy=0.000000 0.000000 0.052347 -> xyz=0.010295 0.000257 0.000000 rpy=0.000000 0.000000 0.049453
- joint joint_13_yaw: origin xyz=0.009983 0.000252 0.000000 rpy=0.000000 0.000000 0.050164 -> xyz=0.010295 0.000245 0.000000 rpy=0.000000 0.000000 0.047336
- joint joint_14_yaw: origin xyz=0.009983 0.000244 0.000000 rpy=0.000000 0.000000 0.048642 -> xyz=0.010295 0.000237 0.000000 rpy=0.000000 0.000000 0.045865
- joint joint_15_yaw: origin xyz=0.009983 0.000239 0.000000 rpy=0.000000 0.000000 0.047706 -> xyz=0.010296 0.000232 0.000000 rpy=0.000000 0.000000 0.044962
- joint joint_16_yaw: origin xyz=0.009983 0.000236 0.000000 rpy=0.000000 0.000000 0.047313 -> xyz=0.010296 0.000230 0.000000 rpy=0.000000 0.000000 0.044583
- joint joint_17_yaw: origin xyz=0.009983 0.000237 0.000000 rpy=0.000000 0.000000 0.047444 -> xyz=0.010296 0.000230 0.000000 rpy=0.000000 0.000000 0.044708
- joint joint_18_yaw: origin xyz=0.009983 0.000239 0.000000 rpy=0.000000 0.000000 0.048104 -> xyz=0.010296 0.000233 0.000000 rpy=0.000000 0.000000 0.045346
- joint joint_19_yaw: origin xyz=0.009983 0.000245 0.000000 rpy=0.000000 0.000000 0.049325 -> xyz=0.010295 0.000238 0.000000 rpy=0.000000 0.000000 0.046525
- joint joint_1_yaw: origin xyz=0.009927 0.000945 0.000000 rpy=0.000000 0.000000 0.186647 -> xyz=0.010230 0.001036 0.000000 rpy=0.000000 0.000000 0.197885
- joint joint_20_yaw: origin xyz=0.009983 0.000254 0.000000 rpy=0.000000 0.000000 0.051167 -> xyz=0.010295 0.000247 0.000000 rpy=0.000000 0.000000 0.048308
- joint joint_21_yaw: origin xyz=0.009982 0.000266 0.000000 rpy=0.000000 0.000000 0.053720 -> xyz=0.010295 0.000259 0.000000 rpy=0.000000 0.000000 0.050788
- joint joint_22_yaw: origin xyz=0.009981 0.000282 0.000000 rpy=0.000000 0.000000 0.057120 -> xyz=0.010294 0.000275 0.000000 rpy=0.000000 0.000000 0.054105
- joint joint_23_yaw: origin xyz=0.009981 0.000303 0.000000 rpy=0.000000 0.000000 0.061553 -> xyz=0.010293 0.000297 0.000000 rpy=0.000000 0.000000 0.058459
- joint joint_24_yaw: origin xyz=0.009979 0.000330 0.000000 rpy=0.000000 0.000000 0.067281 -> xyz=0.010292 0.000325 0.000000 rpy=0.000000 0.000000 0.064130
- joint joint_25_yaw: origin xyz=0.009978 0.000366 0.000000 rpy=0.000000 0.000000 0.074652 -> xyz=0.010291 0.000361 0.000000 rpy=0.000000 0.000000 0.071510
- joint joint_26_yaw: origin xyz=0.009975 0.000411 0.000000 rpy=0.000000 0.000000 0.084130 -> xyz=0.010288 0.000408 0.000000 rpy=0.000000 0.000000 0.081141
- joint joint_27_yaw: origin xyz=0.009972 0.000469 0.000000 rpy=0.000000 0.000000 0.096285 -> xyz=0.010285 0.000470 0.000000 rpy=0.000000 0.000000 0.093740
- joint joint_28_yaw: origin xyz=0.009967 0.000543 0.000000 rpy=0.000000 0.000000 0.111728 -> xyz=0.010279 0.000551 0.000000 rpy=0.000000 0.000000 0.110178
- joint joint_29_yaw: origin xyz=0.009959 0.000635 0.000000 rpy=0.000000 0.000000 0.130858 -> xyz=0.010271 0.000655 0.000000 rpy=0.000000 0.000000 0.131258
- joint joint_2_yaw: origin xyz=0.009940 0.000841 0.000000 rpy=0.000000 0.000000 0.164954 -> xyz=0.010247 0.000903 0.000000 rpy=0.000000 0.000000 0.171003
- joint joint_30_yaw: origin xyz=0.009949 0.000744 0.000000 rpy=0.000000 0.000000 0.153217 -> xyz=0.010259 0.000783 0.000000 rpy=0.000000 0.000000 0.156989
- joint joint_31_yaw: origin xyz=0.009937 0.000860 0.000000 rpy=0.000000 0.000000 0.176356 -> xyz=0.010243 0.000926 0.000000 rpy=0.000000 0.000000 0.184969
- joint joint_32_yaw: origin xyz=0.009925 0.000959 0.000000 rpy=0.000000 0.000000 0.194930 -> xyz=0.010226 0.001054 0.000000 rpy=0.000000 0.000000 0.208501
- joint joint_33_yaw: origin xyz=0.009919 0.001006 0.000000 rpy=0.000000 0.000000 0.202214 -> xyz=0.010218 0.001118 0.000000 rpy=0.000000 0.000000 0.218005
- joint joint_34_yaw: origin xyz=0.009923 0.000982 0.000000 rpy=0.000000 0.000000 0.194930 -> xyz=0.010223 0.001085 0.000000 rpy=0.000000 0.000000 0.208501
- joint joint_35_yaw: origin xyz=0.009934 0.000897 0.000000 rpy=0.000000 0.000000 0.176356 -> xyz=0.010238 0.000973 0.000000 rpy=0.000000 0.000000 0.184969
- joint joint_36_yaw: origin xyz=0.009946 0.000783 0.000000 rpy=0.000000 0.000000 0.153217 -> xyz=0.010255 0.000830 0.000000 rpy=0.000000 0.000000 0.156989
- joint joint_37_yaw: origin xyz=0.009957 0.000670 0.000000 rpy=0.000000 0.000000 0.130858 -> xyz=0.010268 0.000695 0.000000 rpy=0.000000 0.000000 0.131258
- joint joint_38_yaw: origin xyz=0.009965 0.000572 0.000000 rpy=0.000000 0.000000 0.111728 -> xyz=0.010277 0.000583 0.000000 rpy=0.000000 0.000000 0.110178
- joint joint_39_yaw: origin xyz=0.009971 0.000492 0.000000 rpy=0.000000 0.000000 0.096285 -> xyz=0.010283 0.000495 0.000000 rpy=0.000000 0.000000 0.093740
- joint joint_3_yaw: origin xyz=0.009952 0.000725 0.000000 rpy=0.000000 0.000000 0.141725 -> xyz=0.010262 0.000760 0.000000 rpy=0.000000 0.000000 0.143610
- joint joint_40_yaw: origin xyz=0.009975 0.000429 0.000000 rpy=0.000000 0.000000 0.084130 -> xyz=0.010287 0.000427 0.000000 rpy=0.000000 0.000000 0.081141
- joint joint_41_yaw: origin xyz=0.009977 0.000380 0.000000 rpy=0.000000 0.000000 0.074652 -> xyz=0.010290 0.000375 0.000000 rpy=0.000000 0.000000 0.071510
- joint joint_42_yaw: origin xyz=0.009979 0.000341 0.000000 rpy=0.000000 0.000000 0.067281 -> xyz=0.010292 0.000336 0.000000 rpy=0.000000 0.000000 0.064130
- joint joint_43_yaw: origin xyz=0.009980 0.000311 0.000000 rpy=0.000000 0.000000 0.061553 -> xyz=0.010293 0.000305 0.000000 rpy=0.000000 0.000000 0.058459
- joint joint_44_yaw: origin xyz=0.009981 0.000288 0.000000 rpy=0.000000 0.000000 0.057120 -> xyz=0.010294 0.000282 0.000000 rpy=0.000000 0.000000 0.054105
- joint joint_45_yaw: origin xyz=0.009982 0.000271 0.000000 rpy=0.000000 0.000000 0.053720 -> xyz=0.010295 0.000264 0.000000 rpy=0.000000 0.000000 0.050788
- joint joint_46_yaw: origin xyz=0.009982 0.000257 0.000000 rpy=0.000000 0.000000 0.051167 -> xyz=0.010295 0.000251 0.000000 rpy=0.000000 0.000000 0.048308
- joint joint_47_yaw: origin xyz=0.009983 0.000248 0.000000 rpy=0.000000 0.000000 0.049325 -> xyz=0.010295 0.000241 0.000000 rpy=0.000000 0.000000 0.046525
- joint joint_48_yaw: origin xyz=0.009983 0.000241 0.000000 rpy=0.000000 0.000000 0.048104 -> xyz=0.010295 0.000234 0.000000 rpy=0.000000 0.000000 0.045346
- joint joint_49_yaw: origin xyz=0.009983 0.000237 0.000000 rpy=0.000000 0.000000 0.047444 -> xyz=0.010296 0.000231 0.000000 rpy=0.000000 0.000000 0.044708
- joint joint_4_yaw: origin xyz=0.009962 0.000619 0.000000 rpy=0.000000 0.000000 0.120830 -> xyz=0.010273 0.000636 0.000000 rpy=0.000000 0.000000 0.120105
- joint joint_50_yaw: origin xyz=0.009983 0.000236 0.000000 rpy=0.000000 0.000000 0.047313 -> xyz=0.010296 0.000229 0.000000 rpy=0.000000 0.000000 0.044583
- joint joint_51_yaw: origin xyz=0.009983 0.000238 0.000000 rpy=0.000000 0.000000 0.047706 -> xyz=0.010296 0.000231 0.000000 rpy=0.000000 0.000000 0.044962
- joint joint_52_yaw: origin xyz=0.009983 0.000242 0.000000 rpy=0.000000 0.000000 0.048642 -> xyz=0.010295 0.000235 0.000000 rpy=0.000000 0.000000 0.045865
- joint joint_53_yaw: origin xyz=0.009983 0.000249 0.000000 rpy=0.000000 0.000000 0.050164 -> xyz=0.010295 0.000242 0.000000 rpy=0.000000 0.000000 0.047336
- joint joint_54_yaw: origin xyz=0.009982 0.000259 0.000000 rpy=0.000000 0.000000 0.052347 -> xyz=0.010295 0.000252 0.000000 rpy=0.000000 0.000000 0.049453
- joint joint_55_yaw: origin xyz=0.009982 0.000273 0.000000 rpy=0.000000 0.000000 0.055304 -> xyz=0.010294 0.000267 0.000000 rpy=0.000000 0.000000 0.052331
- joint joint_56_yaw: origin xyz=0.009981 0.000292 0.000000 rpy=0.000000 0.000000 0.059193 -> xyz=0.010294 0.000285 0.000000 rpy=0.000000 0.000000 0.056137
- joint joint_57_yaw: origin xyz=0.009980 0.000316 0.000000 rpy=0.000000 0.000000 0.064236 -> xyz=0.010293 0.000310 0.000000 rpy=0.000000 0.000000 0.061108
- joint joint_58_yaw: origin xyz=0.009979 0.000347 0.000000 rpy=0.000000 0.000000 0.070735 -> xyz=0.010291 0.000342 0.000000 rpy=0.000000 0.000000 0.067576
- joint joint_59_yaw: origin xyz=0.009977 0.000387 0.000000 rpy=0.000000 0.000000 0.079095 -> xyz=0.010289 0.000383 0.000000 rpy=0.000000 0.000000 0.076004
- joint joint_5_yaw: origin xyz=0.009968 0.000529 0.000000 rpy=0.000000 0.000000 0.103561 -> xyz=0.010281 0.000536 0.000000 rpy=0.000000 0.000000 0.101422
- joint joint_60_yaw: origin xyz=0.009974 0.000438 0.000000 rpy=0.000000 0.000000 0.089834 -> xyz=0.010287 0.000437 0.000000 rpy=0.000000 0.000000 0.087018
- joint joint_61_yaw: origin xyz=0.009970 0.000504 0.000000 rpy=0.000000 0.000000 0.103561 -> xyz=0.010282 0.000508 0.000000 rpy=0.000000 0.000000 0.101422
- joint joint_62_yaw: origin xyz=0.009964 0.000587 0.000000 rpy=0.000000 0.000000 0.120830 -> xyz=0.010275 0.000600 0.000000 rpy=0.000000 0.000000 0.120105
- joint joint_63_yaw: origin xyz=0.009955 0.000688 0.000000 rpy=0.000000 0.000000 0.141725 -> xyz=0.010265 0.000716 0.000000 rpy=0.000000 0.000000 0.143610
- joint joint_64_yaw: origin xyz=0.009943 0.000802 0.000000 rpy=0.000000 0.000000 0.164954 -> xyz=0.010251 0.000854 0.000000 rpy=0.000000 0.000000 0.171003
- joint joint_65_yaw: origin xyz=0.009930 0.000914 0.000000 rpy=0.000000 0.000000 0.186647 -> xyz=0.010234 0.000995 0.000000 rpy=0.000000 0.000000 0.197885
- joint joint_66_yaw: origin xyz=0.009921 0.000991 0.000000 rpy=0.000000 0.000000 0.200333 -> xyz=0.010220 0.001097 0.000000 rpy=0.000000 0.000000 0.215536
- joint joint_6_yaw: origin xyz=0.009973 0.000458 0.000000 rpy=0.000000 0.000000 0.089834 -> xyz=0.010286 0.000459 0.000000 rpy=0.000000 0.000000 0.087018
- joint joint_7_yaw: origin xyz=0.009976 0.000403 0.000000 rpy=0.000000 0.000000 0.079095 -> xyz=0.010289 0.000399 0.000000 rpy=0.000000 0.000000 0.076004
- joint joint_8_yaw: origin xyz=0.009978 0.000359 0.000000 rpy=0.000000 0.000000 0.070735 -> xyz=0.010291 0.000354 0.000000 rpy=0.000000 0.000000 0.067576
- joint joint_9_yaw: origin xyz=0.009980 0.000325 0.000000 rpy=0.000000 0.000000 0.064236 -> xyz=0.010292 0.000319 0.000000 rpy=0.000000 0.000000 0.061108
