Commit message: inserted 3d printer model to visualization

File: examples/sampling_c3/urdf/3d_Printer/3_d_printer.urdf (robot description, URDF)
Before this commit: robot corexy_printer, 4 links, 3 joints
Links:
- removed link toolhead
- removed link xy_gantry
- added link build_plate, mass 1.0; collision box size=0.355 0.355 0.0202; visual box size=0.355 0.355 0.0202
- added link front_left_post, mass 2.0; visual box size=0.04 0.04 0.475
- added link front_right_post, mass 2.0; visual box size=0.04 0.04 0.475
- added link front_top_rail, mass 1.0; visual box size=0.55 0.04 0.04
- added link left_top_rail, mass 1.0; visual box size=0.04 0.537 0.04
- added link print_volume_marker, mass 0.5; visual box size=0.005 0.005 0.345; visual box size=0.005 0.005 0.345
- added link rear_left_post, mass 2.0; visual box size=0.04 0.04 0.475
- added link rear_right_post, mass 2.0; visual box size=0.04 0.04 0.475
- added link rear_top_rail, mass 1.0; visual box size=0.55 0.04 0.04
- added link right_top_rail, mass 1.0; visual box size=0.04 0.537 0.04
- added link x_carriage, mass 1.0; visual box size=0.080 0.11 0.1092
- added link y_beam, mass 2.0; visual box size=0.43 0.028 0.02
- link base_link: mass None -> 15.0; geometry collision box size=0.55 0.537 0.0798; visual box size=0.55 0.537 0.0596
- link z_gantry: mass None -> 3.0; geometry visual box size=0.02 0.457 0.0265; visual box size=0.02 0.457 0.0265
Joints:
- removed joint x_axis
- removed joint y_axis
- removed joint z_axis
- added joint base_to_build_plate: type fixed, parent base_link, child build_plate, origin xyz=0 -0.0856 0.0899 rpy=0 0 0
- added joint base_to_front_left_post: type fixed, parent base_link, child front_left_post, origin xyz=0.255 0.2485 0.0798 rpy=0 0 0
- added joint base_to_front_right_post: type fixed, parent base_link, child front_right_post, origin xyz=0.255 -0.2485 0.0798 rpy=0 0 0
- added joint base_to_front_top_rail: type fixed, parent base_link, child front_top_rail, origin xyz=0 0.2485 0.5348 rpy=0 0 0
- added joint base_to_left_top_rail: type fixed, parent base_link, child left_top_rail, origin xyz=0.255 0 0.5348 rpy=0 0 0
- added joint base_to_print_volume_marker: type fixed, parent base_link, child print_volume_marker, origin xyz=0.175 0.0894 0.0 rpy=0 0 0
- added joint base_to_rear_left_post: type fixed, parent base_link, child rear_left_post, origin xyz=-0.255 0.2485 0.0798 rpy=0 0 0
- added joint base_to_rear_right_post: type fixed, parent base_link, child rear_right_post, origin xyz=-0.255 -0.2485 0.0798 rpy=0 0 0
- added joint base_to_rear_top_rail: type fixed, parent base_link, child rear_top_rail, origin xyz=0 -0.2485 0.5348 rpy=0 0 0
- added joint base_to_right_top_rail: type fixed, parent base_link, child right_top_rail, origin xyz=-0.255 0 0.5348 rpy=0 0 0
- added joint x_axis_joint: type prismatic, parent y_beam, child x_carriage, origin xyz=0 -0.04068 0.001371 rpy=0 0 0, axis 1 0 0, limit lower=-0.175 upper=0.175 effort=100 velocity=0.5
- added joint y_axis_joint: type prismatic, parent z_gantry, child y_beam, origin xyz=0 -0.038875 0 rpy=0 0 0, axis 0 1 0, limit lower=-0.175 upper=0.175 effort=100 velocity=0.5
- added joint z_axis_joint: type prismatic, parent base_link, child z_gantry, origin xyz=0.175 0.175 0.0474 rpy=0 0 0, axis 0 0 1, limit lower=0.0 upper=0.345 effort=100 velocity=0.5

Commit message: added pose matching to visualization

File: examples/sampling_c3/urdf/3d_Printer/3_d_printer.urdf (robot description, URDF)
Before this commit: robot sovol_sv08_simple, 14 links, 13 joints
Joints:
- joint base_to_build_plate: origin xyz=0 -0.0856 0.0899 rpy=0 0 0 -> xyz=0 0 0.0899 rpy=0 0 0
- joint base_to_print_volume_marker: origin xyz=0.175 0.0894 0.0 rpy=0 0 0 -> xyz=0.175 0.175 0.0 rpy=0 0 0
- joint x_axis_joint: limit lower=-0.175 upper=0.175 effort=100 velocity=0.5 -> lower=0 upper=0.350 effort=100 velocity=0.5; origin xyz=0 -0.04068 0.001371 rpy=0 0 0 -> xyz=-0.175 -0.04068 0.001371 rpy=0 0 0
- joint y_axis_joint: limit lower=-0.175 upper=0.175 effort=100 velocity=0.5 -> lower=0 upper=0.350 effort=100 velocity=0.5; origin xyz=0 -0.038875 0 rpy=0 0 0 -> xyz=0 -0.128275 0 rpy=0 0 0

Commit message: Worked on printer sim

File: examples/sampling_c3/urdf/3d_Printer/3_d_printer.urdf (robot description, URDF)
Before this commit: robot sovol_sv08_simple, 14 links, 13 joints
Links:
- link base_link: geometry collision box size=0.55 0.537 0.0596; visual box size=0.55 0.537 0.0596
