Commit message: three d printer sim working

File: examples/sampling_c3/urdf/3d_Printer/3_d_printer.urdf (robot description, URDF)
Before this commit: robot sovol_sv08_simple, 14 links, 13 joints
Joints:
- joint y_axis_joint: origin xyz=0 -0.128275 0 rpy=0 0 0 -> xyz=0 -0.134375 0 rpy=0 0 0

Commit message: fix kinematics evaluation

File: examples/sampling_c3/urdf/3d_Printer/3_d_printer.urdf (robot description, URDF)
Before this commit: robot sovol_sv08_simple, 14 links, 13 joints
Joints:
- joint y_axis_joint: origin xyz=0 -0.134375 0 rpy=0 0 0 -> xyz=0 -0.128275 0 rpy=0 0 0
