Commit message: fixed 3d printer c3 controller, worked on "osc" controller

File: examples/sampling_c3/urdf/3d_Printer/3_d_printer_bed.urdf (robot description, URDF)
Before this commit: robot sovol_sv08_simple, 1 links, 0 joints
Links:
- removed link base_link
- added link ground, mass 15.0; collision box size=0.55 0.537 0.0596; visual box size=0.55 0.537 0.0596
