Commit message: work on ramp

File: examples/sampling_c3/urdf/3d_Printer/3_d_printer_bed.urdf (robot description, URDF)
Before this commit: robot sovol_sv08_simple_bed, 1 links, 0 joints
Links:
- link ground: mass 15.0 -> 1.0; geometry collision box size=0.355 0.355 0.2; visual box size=0.355 0.355 0.2
