Commit message: work on cube sim

File: examples/sampling_c3/urdf/3d_Printer/ramp.urdf (robot description, URDF)
Before this commit: robot ramp, 1 links, 0 joints
Links:
- link ramp_link: geometry collision box size=0.0762 0.0762 0.0508; collision mesh filename=/mnt/data0/three_d_printer/dairlib/examples/sampling_c3/urd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

Commit message: add new ramp

File: examples/sampling_c3/urdf/3d_Printer/ramp.urdf (robot description, URDF)
Before this commit: robot ramp, 1 links, 0 joints
Links:
- link ramp_link: geometry collision box size=0.19 0.01 0.07; collision box size=0.19 0.01 0.07
