Commit message: Add visualization tools for deformable example

File: examples/deform/models/reduced_mpm_point.urdf (robot description, URDF)
Before this commit: robot reduced_model_point, 1 links, 0 joints
Links:
- added link base_link
- added link pt_fake_x
- added link pt_fake_y
Joints:
- added joint x: type prismatic, parent base_link, child pt_fake_x, axis 1 0 0
- added joint y: type prismatic, parent pt_fake_x, child pt_fake_y, axis 0 1 0
- added joint z: type prismatic, parent pt_fake_y, child reduced_model_point, axis 0 0 1
