Commit message: Minimal changes to run code on other computer

File: examples/sampling_c3/urdf/3d_Printer/ramp/new_ramp.urdf (robot description, URDF)
Before this commit: robot ramp, 1 links, 0 joints
Links:
- link ramp_link: geometry collision mesh filename=ramp1.obj scale=0.001 0.001 0.001; collision mesh filename=ramp10.obj scale=0.001 0.001 0.001
