Commit message: Clamp all output EE plans to respect workspace limits

File: examples/sampling_c3/urdf/three_d_printer/three_d_printer_ee_visualization_model.urdf (robot description, URDF)
Before this commit: robot end_effector_simple, 1 links, 0 joints
Links:
- link end_effector_simple: geometry visual sphere radius=0.011
